File: Eagle/focuser-1.6.brd (EAGLE design)
At the start: 52 x 110.2 mm, 50 parts, among them IC1 78xx, J1 J5MM, J10 J5MM, J2 J7MM, J3 J7MM, J4 J5MM, J5 J7MM, J6 J12MM, J7 J7MM, J8 J7MM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

Commit message: PCB fix for 1.6
Parts:
- added J11: J5MM, jumper:05
- J6: value J12MM -> J15MM; device jumper:12 -> jumper:15
- U$1: value MMduino -> ARDUINONANO
- moved J9 2.54 mm to (14.0, 57.8)
- moved J10 1.91 mm to (11.4, 57.8)
- moved J6 1.53 mm to (31.8, 41.1)
- renumbered NANO to U$1
Connections:
- removed net N$25 (its old number): J10.1, U$1.A6
- removed net VCC: 12V.GND@1, PWR.1
- new net N$40: 12V.POWER, PWR.1
- new net N$41: J10.1, U$1.A7
- new net N$42: U$1.A5, U1.5
- net GND: now also 12V.GND@1; no longer 12V.POWER
- net N$12: now also R5.P$1, U$1.D12; no longer J9.1, U$1.A5
- net N$13: now also U$1.A3, U1.12; no longer U$1.A1, U1.10
- net N$15: now also J11.1, U1.11, U1.6; no longer U$1.A2, U1.12
- net N$3: now also J11.2, U$1.D11; no longer U$1.A0, U1.11, U1.6
- net N$32: now also U$1.D7; no longer U$1.D8
- net N$33: now also U$1.D8; no longer U$1.D9
- net N$34: now also U$1.D9; no longer U$1.D10
- net N$36: now also J9.1, U$1.A6; no longer R5.P$1, U$1.A7
- net N$4: now also U$1.A2, U1.10; no longer U$1.A4, U1.5
- net N$5: now also U$1.A4; no longer U$1.A3
- net N$8: now also U$1.D6; no longer U$1.D7
Routing:
- net N$42: track 0.00 -> 41.4 mm
- net N$3: track 52.8 -> 17.3 mm
- net +5: track 56.7 -> 25.1 mm
- net N$12: track 3.17 -> 26.2 mm
- net N$15: track 46.4 -> 67.4 mm
- net VCC: track 16.9 -> 0.00 mm
- net N$40: track 0.00 -> 10.8 mm
- net N$36: track 9.57 -> 3.17 mm
- net N$13: track 41.8 -> 47.2 mm
- net N$31: track 18.7 -> 14.9 mm
- net N$25 (its old number): track 3.44 -> 0.00 mm
- net N$6: track 14.5 -> 11.3 mm
- net N$25: track 17.7 -> 14.5 mm
- net N$41: track 0.00 -> 3.17 mm
- net N$24: track 110.2 -> 113.3 mm
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