File: Eagle/focuser-1.6.sch (EAGLE design)
At the start: 46 parts, among them IC1 78xx, J1 J5MM, J10 J5MM, J2 J7MM, J3 J7MM, J4 J5MM, J5 J7MM, J6 J12MM, J7 J7MM, J8 J7MM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

Commit message: PCB fix for 1.6
Parts:
- added J11: J5MM, jumper:J5MM
- J6: value J12MM -> J15MM; device jumper:J12MM -> jumper:J15MM
- U$1: value MMduino -> ARDUINONANO; NAM Arduino NANO -> (none)
- renumbered NANO to U$1
Connections:
- removed net N$25 (its old number): J10.1, U$1.A6
- removed net VCC: 12V.GND, PWR.1
- new net N$40: 12V.PWR, PWR.1
- new net N$41: J10.1, U$1.A0
- new net N$42: U$1.A2, U1.IN1
- net GND: now also 12V.GND; no longer 12V.PWR
- net N$12: now also R5.1, U$1.D12; no longer J9.1, U$1.A5
- net N$13: now also U$1.A4, U1.IN4; no longer U$1.A1, U1.IN3
- net N$15: now also J11.1, U1.ENA, U1.ENB; no longer U$1.A2, U1.IN4
- net N$3: now also J11.2, U$1.D11; no longer U$1.A0, U1.ENA, U1.ENB
- net N$32: now also U$1.D7; no longer U$1.D8
- net N$33: now also U$1.D8; no longer U$1.D9
- net N$34: now also U$1.D9; no longer U$1.D10
- net N$36: now also J9.1, U$1.A1; no longer R5.1, U$1.A7
- net N$4: now also U$1.A5, U1.IN3; no longer U$1.A4, U1.IN1
- net N$8: now also U$1.D6; no longer U$1.D7
Other:
- moved on the sheet: ., J10, J9
