File: Eagle/focuser.sch (EAGLE design)
At the start: 46 parts, among them IC1 78xx, J1 J5MM, J10 J5MM, J2 J7MM, J3 J7MM, J4 J5MM, J5 J7MM, J6 J12MM, J7 J7MM, J8 J7MM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

Commit message: Production final refactor
Parts:
- U$1: value MMduino -> ARDUINONANO; NAM Arduino NANO -> (none)
- renumbered NANO to U$1
Connections:
- removed net N$15: U$1.A2, U1.IN4
- removed net N$25: J10.1, U$1.A6
- removed net N$4 (its old number): U$1.A4, U1.IN1
- new net N$13: U$1.A5, U1.IN4
- new net N$41: J9.2, U$1.A7
- new net N$42: U$1.A3, U1.IN1
- net N$12: now also J10.2, U$1.A6; no longer J9.1, U$1.A5
- net N$3: now also U$1.D6; no longer U$1.A0
- net N$31: now also J10.1; no longer J10.2
- net N$36: now also U$1.A0; no longer U$1.A7
- net N$40: now also J9.1; no longer J9.2
- net N$5: now also U$1.A4; no longer U$1.A3
Other:
- moved on the sheet: J10, J9

Commit message: PCB fix for 1.6
Parts:
- NANO: value ARDUINONANO -> MMduino; NAM (none) -> Arduino NANO
- renumbered U$1 to NANO
Connections:
- removed net N$13 (its old number): NANO.A5, U1.IN4
- removed net N$41: J9.2, NANO.A7
- removed net N$42: NANO.A3, U1.IN1
- new net N$15: NANO.A2, U1.IN4
- new net N$25: J10.1, NANO.A6
- new net N$4: NANO.A4, U1.IN1
- net N$12: now also J9.1, NANO.A5; no longer J10.2, NANO.A6
- net N$3: now also NANO.A0; no longer NANO.D6
- net N$31: now also J10.2; no longer J10.1
- net N$36: now also NANO.A7; no longer NANO.A0
- net N$40: now also J9.2; no longer J9.1
- net N$5: now also NANO.A3; no longer NANO.A4
Other:
- moved on the sheet: J10, J9
