File: Eagle/focuser.sch (EAGLE design)
At the start: 46 parts, among them IC1 78xx, J1 J5MM, J10 J5MM, J2 J7MM, J3 J7MM, J4 J5MM, J5 J7MM, J6 J12MM, J7 J7MM, J8 J7MM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

Commit message: Focuser 2.0
Parts:
- removed ...: (no value), SparkFun:JUMPER-2PTH
- added ...1: (no value), SparkFun:JUMPER-2PTH
- added ..1: JUMPER-3PTH, SparkFun:JUMPER-3PTH
- added J11: J5MM, jumper:J5MM
Connections:
- removed net N$30: C3.+, J8.1, R1.2, TEMP.5
- new net N$41: ..1.1, NANO.D10
- new net N$42: ...3, NANO.D11
- new net N$43: ...2, NANO.D12
- new net N$44: C5.+, J11.2, NANO.VIN
- new net N$45: J6.1, J8.2, NANO.+5V
- net +5: now also C3.+, J8.1, R1.2, TEMP.5; no longer J6.1, J8.2, NANO.+5V
- net N$18: now also NANO.D6; no longer NANO.D4
- net N$24: now also NANO.D7; no longer NANO.D3
- net N$31: now also ...1; no longer ..2
- net N$32: now also ...1.2, NANO.D4; no longer ...3, NANO.D8
- net N$33: now also ...1.1, NANO.D5; no longer ...2, NANO.D9
- net N$34: now also ..1.3, NANO.D8; no longer ...1, NANO.D10
- net N$35: now also ..1.2, NANO.D9; no longer NANO.D5, R2.1
- net N$6: now also ..2; no longer ....2
- net N$8: now also NANO.D3, R2.1; no longer ....1, NANO.D7
- net N$9: now also J11.1; no longer C5.+, NANO.VIN
Other:
- moved on the sheet: ., .., J8, R2

Commit message: Focuser 2.0 - PCB
Parts:
- removed ...1: (no value), SparkFun:JUMPER-2PTH
- added ..2: JUMPER-3PTH, SparkFun:JUMPER-3PTH
Connections:
- removed net N$40: ..3, J9.2
- removed net VCC: 12V.GND, PWR.1
- new net N$30: 12V.PWR, PWR.1
- new net N$46: ..2.1, ..3, J9.2
- net GND: now also 12V.GND; no longer 12V.PWR
- net N$32: now also ..2.3; no longer ...1.2
- net N$33: now also ..2.2; no longer ...1.1
Changed lines of the file:
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@@
 <part name="J9" library="jumper" deviceset="J" device="5MM" value="J5MM"/>
 <part name="J10" library="jumper" deviceset="J" device="5MM" value="J5MM"/>
-<part name="...1" library="SparkFun" deviceset="JUMPER-2" device="PTH"/>
 <part name="..1" library="SparkFun" deviceset="JUMPER-3" device="PTH" value=""/>
 <part name="J11" library="jumper" deviceset="J" device="5MM" value="J5MM"/>
+<part name="..2" library="SparkFun" deviceset="JUMPER-3" device="PTH" value=""/>
 </parts>
 <sheets>
@@
 <instance part="J9" gate="1" x="71.12" y="38.1"/>
 <instance part="J10" gate="1" x="68.58" y="33.02"/>
-<instance part="...1" gate="A" x="15.24" y="35.56" rot="R90"/>
 <instance part="..1" gate="G$1" x="15.24" y="22.86" rot="R90"/>
 <instance part="J11" gate="1" x="71.12" y="93.98" rot="R270"/>
+<instance part="..2" gate="G$1" x="15.24" y="33.02" rot="R90"/>
 </instances>
 <busses>
@@
 <pinref part="C1" gate="G$1" pin="2"/>
 <pinref part="GND9" gate="1" pin="GND"/>
-</segment>
-<segment>
-<pinref part="12V" gate="G$1" pin="PWR"/>
-<wire x1="-2.54" y1="109.22" x2="12.7" y2="109.22" width="0.1524" layer="91"/>
-<pinref part="GND10" gate="1" pin="GND"/>
-<wire x1="12.7" y1="109.22" x2="12.7" y2="96.52" width="0.1524" layer="91"/>
 </segment>
 <segment>
@@
 <wire x1="17.78" y1="1.016" x2="12.446" y2="1.016" width="0.1524" layer="91"/>
 </segment>
+<segment>
+<pinref part="GND10" gate="1" pin="GND"/>
+<wire x1="12.7" y1="96.52" x2="12.7" y2="104.14" width="0.1524" layer="91"/>
+<pinref part="12V" gate="G$1" pin="GND"/>
+<wire x1="12.7" y1="104.14" x2="-2.54" y2="104.14" width="0.1524" layer="91"/>
+</segment>
 </net>
 <net name="VCC2" class="1">
@@
 <wire x1="154.94" y1="17.78" x2="154.94" y2="33.02" width="0.1524" layer="91"/>
 <junction x="154.94" y="33.02"/>
-</segment>
-</net>
-<net name="VCC" class="1">
-<segment>
-<pinref part="12V" gate="G$1" pin="GND"/>
-<wire x1="-2.54" y1="104.14" x2="17.78" y2="104.14" width="0.1524" layer="91"/>
-<pinref part="PWR" gate="A" pin="1"/>
-<wire x1="17.78" y1="104.14" x2="17.78" y2="111.76" width="0.1524" layer="91"/>
 </segment>
 </net>
@@
 </segment>
 </net>
-<net name="N$40" class="0">
-<segment>
-<pinref part="J9" gate="1" pin="2"/>
-<wire x1="76.2" y1="38.1" x2="76.2" y2="0" width="0.1524" layer="91"/>
-<wire x1="76.2" y1="0" x2="20.32" y2="0" width="0.1524" layer="91"/>
-<wire x1="20.32" y1="0" x2="20.32" y2="12.7" width="0.1524" layer="91"/>
-<pinref part="." gate="G$1" pin="3"/>
-<wire x1="20.32" y1="12.7" x2="17.78" y2="12.7" width="0.1524" layer="91"/>
-</segment>
-</net>
 <net name="N$8" class="0">
 <segment>
@@
 <net name="N$32" class="0">
 <segment>
-<pinref part="...1" gate="A" pin="2"/>
 <wire x1="17.78" y1="38.1" x2="18.796" y2="38.1" width="0.1524" layer="91"/>
 <wire x1="18.796" y1="38.1" x2="18.796" y2="53.34" width="0.1524" layer="91"/>
 <pinref part="NANO" gate="G$1" pin="D4"/>
 <wire x1="18.796" y1="53.34" x2="27.94" y2="53.34" width="0.1524" layer="91"/>
+<pinref part="..2" gate="G$1" pin="3"/>
 </segment>
 </net>
 <net name="N$33" class="0">
 <segment>
-<pinref part="...1" gate="A" pin="1"/>
 <wire x1="17.78" y1="35.56" x2="20.32" y2="35.56" width="0.1524" layer="91"/>
 <wire x1="20.32" y1="35.56" x2="20.32" y2="48.26" width="0.1524" layer="91"/>
 <pinref part="NANO" gate="G$1" pin="D5"/>
 <wire x1="20.32" y1="48.26" x2="27.94" y2="48.26" width="0.1524" layer="91"/>
-</segment>
-</net>
-<net name="N$34" class="0">
-<segment>
-<pinref part="..1" gate="G$1" pin="3"/>
-<wire x1="17.78" y1="27.94" x2="17.78" y2="33.02" width="0.1524" layer="91"/>
-<pinref part="NANO" gate="G$1" pin="D8"/>
-<wire x1="17.78" y1="33.02" x2="27.94" y2="33.02" width="0.1524" layer="91"/>
-</segment>
-</net>
-<net name="N$35" class="0">
-<segment>
-<pinref part="..1" gate="G$1" pin="2"/>
-<wire x1="17.78" y1="25.4" x2="20.32" y2="25.4" width="0.1524" layer="91"/>
-<wire x1="20.32" y1="25.4" x2="20.32" y2="27.94" width="0.1524" layer="91"/>
-<pinref part="NANO" gate="G$1" pin="D9"/>
-<wire x1="20.32" y1="27.94" x2="27.94" y2="27.94" width="0.1524" layer="91"/>
+<pinref part="..2" gate="G$1" pin="2"/>
 </segment>
 </net>
@@
 </segment>
 </net>
+<net name="N$30" class="0">
+<segment>
+<pinref part="12V" gate="G$1" pin="PWR"/>
+<wire x1="-2.54" y1="109.22" x2="17.78" y2="109.22" width="0.1524" layer="91"/>
+<pinref part="PWR" gate="A" pin="1"/>
+<wire x1="17.78" y1="109.22" x2="17.78" y2="111.76" width="0.1524" layer="91"/>
+</segment>
+</net>
+<net name="N$34" class="0">
+<segment>
+<pinref part="..1" gate="G$1" pin="2"/>
+<wire x1="17.78" y1="25.4" x2="25.4" y2="25.4" width="0.1524" layer="91"/>
+<wire x1="25.4" y1="25.4" x2="25.4" y2="27.94" width="0.1524" layer="91"/>
+<pinref part="NANO" gate="G$1" pin="D9"/>
+<wire x1="25.4" y1="27.94" x2="27.94" y2="27.94" width="0.1524" layer="91"/>
+</segment>
+</net>
+<net name="N$35" class="0">
+<segment>
+<pinref part="..1" gate="G$1" pin="3"/>
+<wire x1="17.78" y1="27.94" x2="22.86" y2="27.94" width="0.1524" layer="91"/>
+<wire x1="22.86" y1="27.94" x2="22.86" y2="33.02" width="0.1524" layer="91"/>
+<pinref part="NANO" gate="G$1" pin="D8"/>
+<wire x1="22.86" y1="33.02" x2="27.94" y2="33.02" width="0.1524" layer="91"/>
+</segment>
+</net>
+<net name="N$46" class="0">
+<segment>
+<pinref part="..2" gate="G$1" pin="1"/>
+<wire x1="17.78" y1="33.02" x2="20.32" y2="33.02" width="0.1524" layer="91"/>
+<pinref part="J9" gate="1" pin="2"/>
+<wire x1="76.2" y1="38.1" x2="76.2" y2="0" width="0.1524" layer="91"/>
+<wire x1="76.2" y1="0" x2="20.32" y2="0" width="0.1524" layer="91"/>
+<wire x1="20.32" y1="0" x2="20.32" y2="12.7" width="0.1524" layer="91"/>
+<pinref part="." gate="G$1" pin="3"/>
+<wire x1="20.32" y1="12.7" x2="17.78" y2="12.7" width="0.1524" layer="91"/>
+<wire x1="20.32" y1="33.02" x2="20.32" y2="12.7" width="0.1524" layer="91"/>
+<junction x="20.32" y="12.7"/>
+</segment>
+</net>
 </nets>
 </sheet>
 </sheets>
+<errors>
+</errors>
 </schematic>
 </drawing>

Commit message: Arduino / Eagle updates
Parts:
- removed .: JUMPER-3PTH, SparkFun:JUMPER-3PTH
- C3, C5: device SparkFun:CAP_POLPTH1 -> resistor:CPOL-EUE2-4
- J10, J11: value J5MM -> J7MM; device jumper:J5MM -> jumper:J7MM
- SG1: device buzzer:F/QMBIII -> buzzer2:F/QMBIII
Connections:
- removed net N$18 (its old number): CONTROL.2, MANUAL.2, NANO.D6
- removed net N$31 (its old number): ...1, J10.2
- removed net N$36: NANO.A7, R5.1
- removed net N$46: ..2.1, ..3, J9.2
- new net N$33: NANO.D4, R2.1
- new net N$41: J10.2, NANO.A1
- net GND: now also ...1, 12V.GNDBREAK; no longer ..1
- net N$12: now also NANO.A0, R5.1; no longer J9.1, NANO.A5
- net N$13: now also NANO.A5; no longer NANO.A1
- net N$15: now also NANO.A4; no longer NANO.A2
- net N$25: now also ...3, NANO.D12; no longer J10.1, NANO.A6
- net N$3: now also J9.2; no longer NANO.A0
- net N$32: now also NANO.D3; no longer NANO.D4
- net N$35: now also ..2.1, NANO.D6; no longer ..1.3, NANO.D8
- net N$4: now also NANO.A2; no longer NANO.A4
- net N$42: now also J9.1; no longer ...3
- net N$43: now also ..1.3, J10.1; no longer ...2, NANO.D12
- net N$6: now also ...2; no longer ..2
- net N$8: now also CONTROL.2, MANUAL.2, NANO.D8; no longer NANO.D3, R2.1
Other:
- moved on the sheet: .., ..1, ..2, CONTROL, J10, J9, MANUAL, R2, R5, SG1
