File: Eagle/focuser.sch (EAGLE design)
At the start: 14 parts, among them IC1 L293D, IC2 L293D, IC3 PCF8574P

Commit message: Work continues... VB script update
Connections:
- new net N$10: U$1.6
- new net N$11: U$1.5
- new net N$12: U$1.3
- new net N$13: U$1.11
- new net N$14: U$1.13
- new net N$3: U$1.A3, U$7.STEP
- new net N$4: U$1.A2, U$7.DIR
- new net N$5: U$1.A1, U$6.STEP
- new net N$6: U$1.A0, U$6.DIR
- new net N$7: U$1.10, U$7.EN
- new net N$8: U$1.9, U$6.EN
Changed lines of the file:
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@@
 <instance part="..2" gate="G$1" x="-33.02" y="45.72" rot="R90"/>
 <instance part="U$1" gate="G$1" x="116.84" y="81.28"/>
-<instance part="U$6" gate="G$1" x="182.88" y="38.1"/>
-<instance part="U$7" gate="G$1" x="182.88" y="96.52"/>
-<instance part="U$8" gate="G$1" x="40.64" y="81.28"/>
+<instance part="U$6" gate="G$1" x="182.88" y="43.18"/>
+<instance part="U$7" gate="G$1" x="182.88" y="99.06"/>
+<instance part="U$8" gate="G$1" x="20.32" y="81.28"/>
 <instance part="IC1" gate="G$1" x="190.5" y="160.02" rot="R90"/>
 <instance part="IC2" gate="G$1" x="190.5" y="210.82" rot="R90"/>
@@
 <net name="N$1" class="0">
 <segment>
-<pinref part="U$8" gate="G$1" pin="A5"/>
-<wire x1="48.26" y1="30.48" x2="48.26" y2="25.4" width="0.1524" layer="91"/>
-<wire x1="48.26" y1="25.4" x2="83.82" y2="25.4" width="0.1524" layer="91"/>
+<wire x1="27.94" y1="25.4" x2="83.82" y2="25.4" width="0.1524" layer="91"/>
 <pinref part="U$1" gate="G$1" pin="A5"/>
 <wire x1="83.82" y1="25.4" x2="124.46" y2="25.4" width="0.1524" layer="91"/>
@@
 <wire x1="83.82" y1="139.7" x2="83.82" y2="25.4" width="0.1524" layer="91"/>
 <junction x="83.82" y="25.4"/>
+<pinref part="U$8" gate="G$1" pin="A5"/>
+<wire x1="27.94" y1="30.48" x2="27.94" y2="25.4" width="0.1524" layer="91"/>
 </segment>
 </net>
 <net name="N$2" class="0">
 <segment>
-<pinref part="U$8" gate="G$1" pin="A4"/>
-<wire x1="43.18" y1="30.48" x2="43.18" y2="22.86" width="0.1524" layer="91"/>
-<wire x1="43.18" y1="22.86" x2="81.28" y2="22.86" width="0.1524" layer="91"/>
+<wire x1="22.86" y1="22.86" x2="81.28" y2="22.86" width="0.1524" layer="91"/>
 <pinref part="U$1" gate="G$1" pin="A4"/>
 <wire x1="81.28" y1="22.86" x2="119.38" y2="22.86" width="0.1524" layer="91"/>
@@
 <wire x1="81.28" y1="142.24" x2="81.28" y2="22.86" width="0.1524" layer="91"/>
 <junction x="81.28" y="22.86"/>
+<pinref part="U$8" gate="G$1" pin="A4"/>
+<wire x1="22.86" y1="22.86" x2="22.86" y2="30.48" width="0.1524" layer="91"/>
 </segment>
 </net>
+<net name="N$3" class="0">
+<segment>
+<pinref part="U$1" gate="G$1" pin="A3"/>
+<pinref part="U$7" gate="G$1" pin="STEP"/>
+<wire x1="137.16" y1="81.28" x2="167.64" y2="81.28" width="0.1524" layer="91"/>
+</segment>
+</net>
+<net name="N$4" class="0">
+<segment>
+<pinref part="U$1" gate="G$1" pin="A2"/>
+<pinref part="U$7" gate="G$1" pin="DIR"/>
+<wire x1="137.16" y1="76.2" x2="167.64" y2="76.2" width="0.1524" layer="91"/>
+</segment>
+</net>
+<net name="N$5" class="0">
+<segment>
+<pinref part="U$1" gate="G$1" pin="A1"/>
+<wire x1="137.16" y1="71.12" x2="162.56" y2="71.12" width="0.1524" layer="91"/>
+<wire x1="162.56" y1="71.12" x2="162.56" y2="25.4" width="0.1524" layer="91"/>
+<pinref part="U$6" gate="G$1" pin="STEP"/>
+<wire x1="162.56" y1="25.4" x2="167.64" y2="25.4" width="0.1524" layer="91"/>
+</segment>
+</net>
+<net name="N$6" class="0">
+<segment>
+<pinref part="U$1" gate="G$1" pin="A0"/>
+<wire x1="137.16" y1="66.04" x2="160.02" y2="66.04" width="0.1524" layer="91"/>
+<wire x1="160.02" y1="66.04" x2="160.02" y2="20.32" width="0.1524" layer="91"/>
+<pinref part="U$6" gate="G$1" pin="DIR"/>
+<wire x1="160.02" y1="20.32" x2="167.64" y2="20.32" width="0.1524" layer="91"/>
+</segment>
+</net>
+<net name="N$7" class="0">
+<segment>
+<pinref part="U$1" gate="G$1" pin="10"/>
+<wire x1="137.16" y1="45.72" x2="157.48" y2="45.72" width="0.1524" layer="91"/>
+<wire x1="157.48" y1="45.72" x2="157.48" y2="111.76" width="0.1524" layer="91"/>
+<pinref part="U$7" gate="G$1" pin="EN"/>
+<wire x1="157.48" y1="111.76" x2="167.64" y2="111.76" width="0.1524" layer="91"/>
+</segment>
+</net>
+<net name="N$8" class="0">
+<segment>
+<pinref part="U$1" gate="G$1" pin="9"/>
+<wire x1="91.44" y1="45.72" x2="88.9" y2="45.72" width="0.1524" layer="91"/>
+<wire x1="88.9" y1="45.72" x2="88.9" y2="15.24" width="0.1524" layer="91"/>
+<wire x1="88.9" y1="15.24" x2="154.94" y2="15.24" width="0.1524" layer="91"/>
+<wire x1="154.94" y1="15.24" x2="154.94" y2="55.88" width="0.1524" layer="91"/>
+<pinref part="U$6" gate="G$1" pin="EN"/>
+<wire x1="154.94" y1="55.88" x2="167.64" y2="55.88" width="0.1524" layer="91"/>
+</segment>
+</net>
+<net name="N$10" class="0">
+<segment>
+<pinref part="U$1" gate="G$1" pin="6"/>
+<wire x1="91.44" y1="60.96" x2="76.2" y2="60.96" width="0.1524" layer="91"/>
+<wire x1="76.2" y1="60.96" x2="76.2" y2="2.54" width="0.1524" layer="91"/>
+</segment>
+</net>
+<net name="N$11" class="0">
+<segment>
+<pinref part="U$1" gate="G$1" pin="5"/>
+<wire x1="91.44" y1="66.04" x2="73.66" y2="66.04" width="0.1524" layer="91"/>
+<wire x1="73.66" y1="66.04" x2="73.66" y2="2.54" width="0.1524" layer="91"/>
+</segment>
+</net>
+<net name="N$12" class="0">
+<segment>
+<pinref part="U$1" gate="G$1" pin="3"/>
+<wire x1="91.44" y1="76.2" x2="71.12" y2="76.2" width="0.1524" layer="91"/>
+<wire x1="71.12" y1="76.2" x2="71.12" y2="2.54" width="0.1524" layer="91"/>
+</segment>
+</net>
+<net name="N$13" class="0">
+<segment>
+<pinref part="U$1" gate="G$1" pin="11"/>
+<wire x1="137.16" y1="50.8" x2="139.7" y2="50.8" width="0.1524" layer="91"/>
+<wire x1="139.7" y1="50.8" x2="139.7" y2="17.78" width="0.1524" layer="91"/>
+<wire x1="139.7" y1="17.78" x2="78.74" y2="17.78" width="0.1524" layer="91"/>
+<wire x1="78.74" y1="17.78" x2="78.74" y2="2.54" width="0.1524" layer="91"/>
+</segment>
+</net>
+<net name="N$14" class="0">
+<segment>
+<pinref part="U$1" gate="G$1" pin="13"/>
+<wire x1="137.16" y1="60.96" x2="142.24" y2="60.96" width="0.1524" layer="91"/>
+<wire x1="142.24" y1="60.96" x2="142.24" y2="-2.54" width="0.1524" layer="91"/>
+<wire x1="142.24" y1="-2.54" x2="-20.32" y2="-2.54" width="0.1524" layer="91"/>
+<wire x1="-20.32" y1="-2.54" x2="-20.32" y2="0" width="0.1524" layer="91"/>
+</segment>
+</net>

Commit message: Schematic update
Parts:
- removed .., ..1, ..2: JUMPER-3PTH, SparkFun:JUMPER-3PTH
- removed IC3: PCF8574P, micro-philips:PCF8574P
- added 12V1, 12V2, 12V3, 12V4, 12V5, 12V6: Jack 5.5/2.1, SparkFun:POWER_JACKCOMBO
- added C1: 1000u, SparkFun:CAP_POLPTH4
- added C10, C8: 10u, SparkFun:CAP_POLPTH2
- added C2, C3, C4, C5, C6, C7, C9: 100n, SparkFun:CAPPTH1
- added D1, D2: (no value), SparkFun:DIODE1N4148
- added F1, F2, F3, F4, F5, F6, F7: PTCPTH, SparkFun:PTCPTH
- added IC4: L293D, st-microelectronics:L293D
- added IC5: 7809, SparkFun:V_REG_78XXSINK
- added IC6: ULN2003AN, uln-udn:ULN2003AN
- added J1, J2, J3, J4: POWER_JACKRCA, SparkFun:POWER_JACKRCA
- added Q1, Q2, Q3, Q4: IRF540, transistor-fet:IRF540
- added R1, R7, R8, R9: 100, SparkFun:RESISTORPTH1
- added R10, R11, R12, R3, R4, R5, R6: 3k3, SparkFun:RESISTORPTH1
- added TEMP1, TEMP2: Jack 3.5mm, SparkFun:AUDIO-JACKPTH
- added U$10, U$14: DCDC-5V, jolo-lib:DCDC-STEPDOWN
- added U$11, U$12, U$13, U$15, U$9: RELAYPTH, SparkFun:RELAYPTH
- added U$16: I2C, SparkFun:RJ9PTH
- added X1, X2: (no value), SparkFun:DB9
- IC2: MPN (none) -> L293D; OC_FARNELL (none) -> 9589619; OC_NEWARK (none) -> 56P8249
- U$6: value A4988-MODULE -> SW motor; device jolo-lib:A4988-MODULE -> SparkFun:RJ9PTH
- U$7: value A4988-MODULE -> Hand control; device jolo-lib:A4988-MODULE -> SparkFun:RJ9PTH
Connections:
- removed net GND: SG1.+
- new net +12V: 12V.PWR, 12V5.PWR, C1.+, C2.1, C3.1, C9.1, F1.1, F2.1, F3.2, IC5.IN, IC6.CD+, J1.PWR, J2.PWR, J3.PWR, J4.PWR, U$11.COIL2, U$11.MAIN, U$12.COIL2, U$12.MAIN, U$13.COIL2, U$13.MAIN, U$15.COIL2, U$9.COIL2, U$9.MAIN
- new net +5V: C10.+, C4.2, C5.2, C8.+, IC1.VCC2, IC2.VCC2, IC4.VCC2, R10.2, R11.2, R12.2, TEMP.5, TEMP1.5, TEMP2.5, U$1.VCC2, U$10.VCCOUT, U$16.4, U$7.4, U$8.VCC2
- new net 3.3V: C7.1, IC4.VCC1, IC5.OUT
- new net AGND: 12V.GND, 12V.GNDBREAK, 12V1.GND, 12V1.GNDBREAK, 12V2.GND, 12V2.GNDBREAK, 12V3.GND, 12V3.GNDBREAK, 12V4.GND, 12V4.GNDBREAK, 12V5.GND, 12V5.GNDBREAK, 12V6.GND, 12V6.GNDBREAK, C1.-, C2.2, C3.2, C6.2, C7.2, C9.2, IC1.GND1, IC1.GND2, IC1.GND3, IC1.GND4, IC2.GND1, IC2.GND2, IC2.GND3, IC2.GND4, IC4.GND1, IC4.GND2, IC4.GND3, IC4.GND4, IC5.GND, Q1.S, Q2.S, Q3.S, Q4.S, R3.2, R4.2, R5.2, R6.2, X1.9, X2.9
- new net DGND: C10.-, C4.1, C5.1, C8.-, SG1.+, TEMP.1, TEMP1.1, TEMP2.1, U$1.GND, U$10.GNDIN, U$10.GNDOUT, U$14.GNDIN, U$14.GNDOUT, U$16.1, U$7.1, U$8.GND
- new net N$15: IC2.2Y, X2.1
- new net N$16: IC1.2Y, X1.1
- new net N$17: D1.C, D2.C, R2.1
- new net N$18: IC6.I1, U$8.8
- new net N$19: IC1.2A, U$1.2
- new net N$20: IC1.1A, U$1.4
- new net N$21: IC2.3A, U$1.8
- new net N$22: IC2.4A, U$1.7
- new net N$23: IC6.I2, U$8.7
- new net N$25: IC6.I3, U$8.6
- new net N$27: IC6.I4, U$8.5
- new net N$28: U$7.2, U$8.A0
- new net N$30: IC4.1-2EN, IC4.3-4EN, U$8.9
- new net N$35: J1.GND, J1.GNDBREAK, Q1.D
- new net N$36: J2.GND, J2.GNDBREAK, Q2.D
- new net N$37: 12V6.PWR, U$15.NO
- new net N$38: J3.GND, J3.GNDBREAK, Q3.D
- new net N$39: Q4.G, R6.1, R9.1
- new net N$40: Q3.G, R5.1, R8.1
- new net N$41: Q2.G, R4.1, R7.1
- new net N$42: Q1.G, R1.1, R3.1
- new net N$43: 12V1.PWR, F4.1
- new net N$45: IC4.3Y, U$6.4
- new net N$46: D1.A, U$8.13
- new net N$47: R9.2, U$1.11
- new net N$48: R8.2, U$1.3
- new net N$49: R7.2, U$1.5
- new net N$50: R1.2, U$1.6
- new net N$51: U$6.3
- new net N$52: 12V2.PWR, F5.1
- new net N$54: IC6.O5, U$9.COIL1
- new net N$55: IC6.O4, U$11.COIL1
- new net N$56: IC6.O3, U$12.COIL1
- new net N$57: IC6.O2, U$13.COIL1
- new net N$58: C6.1, F3.1, IC1.VCC1, IC2.VCC1, X1.5, X2.5
- new net N$59: R12.1, TEMP.2, U$8.A1
- new net N$60: 12V3.PWR, F6.1
- new net N$61: 12V4.PWR, F7.1
- new net N$62: F7.2, U$13.NO
- new net N$63: IC6.O1, U$15.COIL1
- new net N$64: J4.GND, J4.GNDBREAK, Q4.D
- new net N$65: R11.1, TEMP1.2, U$8.A2
- new net N$66: F6.2, U$12.NO
- new net N$67: F5.2, U$11.NO
- new net N$68: F4.2, U$9.NO
- new net N$69: F1.2, U$10.VCCIN
- new net N$70: F2.2, U$14.VCCIN
- new net N$71: R10.1, TEMP2.2, U$8.A3
- new net N$73: IC2.3Y, X2.4
- new net N$74: IC4.4A, U$8.11
- new net N$75: IC4.3A, U$8.10
- new net N$9: IC1.4A, U$1.A2
- new net V+: U$14.VCCOUT, U$15.MAIN
- net N$1: now also U$16.2; no longer IC3.SCL
- net N$10: now also IC2.1A, U$1.A1; no longer U$1.6
- net N$11: now also IC2.2A, U$1.A0; no longer U$1.5
- net N$12: now also IC2.1-2EN, IC2.3-4EN, U$1.10; no longer U$1.3
- net N$13: now also IC2.1Y, X2.2; no longer U$1.11
- net N$14: now also D2.A
- net N$2: now also U$16.3; no longer IC3.SDA
- net N$3: now also IC1.3A; no longer U$7.STEP
- net N$4: now also IC2.4Y, X2.3; no longer U$1.A2, U$7.DIR
- net N$5: now also IC1.1Y, X1.2; no longer U$1.A1, U$6.STEP
- net N$6: now also IC1.4Y, X1.3; no longer U$1.A0, U$6.DIR
- net N$7: now also IC1.3Y, X1.4; no longer U$1.10, U$7.EN
- net N$8: now also IC1.3-4EN; no longer U$6.EN
Other:
- moved on the sheet: 12V, IC1, IC2, R2, SG1, TEMP

Commit message: no message
Parts:
- removed C4: 100n, SparkFun:CAPPTH1
- removed D1, D2: (no value), SparkFun:DIODE1N4148
- removed U$1, U$8: ARDUINO-MINI-PRO, jolo-lib:ARDUINO-MINI-PRO
- added 5V: Jack 5.5/2.1, SparkFun:POWER_JACKCOMBO
- added JP1: (no value), pinhead:PINHD-1X10
- added R13, R14: 2k, SparkFun:RESISTORPTH1
- added R15, R16: 1k, SparkFun:RESISTORPTH1
- added U1: ARDUINO-MEGAFULL, SparkFun-Boards:ARDUINO-MEGAFULL
- IC5: device SparkFun:V_REG_78XXSINK -> SparkFun:V_REG_78XXSIDE
Connections:
- removed net N$17: D1.C, D2.C, R2.1
- removed net N$48: R8.2, U$1.3
- removed net N$49: R7.2, U$1.5
- removed net N$50: R1.2, U$1.6
- new net N$29: IC6.I2, U1.51
- new net N$31: IC4.3A, U1.45
- new net N$32: R7.2, U1.11
- new net N$33: R8.2, U1.10
- new net N$34: U$7.2, U1.A0(RX0)
- new net N$44: U$7.3
- new net N$53: JP1.2, U1.34
- new net N$72: JP1.3, U1.35
- new net N$76: JP1.6, U1.38
- new net N$77: JP1.7, U1.39
- new net N$78: JP1.8, U1.40
- new net N$79: JP1.9, U1.41
- net +12V: now also R14.1
- net +5V: now also 5V.PWR, C5.1, JP1.1, U1.5V@0, U1.5V@1, U1.5V@2; no longer C4.2, C5.2, U$1.VCC2, U$8.VCC2
- net DGND: now also 5V.GND, 5V.GNDBREAK, C5.2, JP1.10, R15.2, R16.2, U1.GND@0, U1.GND@1, U1.GND@2, U1.GND@3, U1.GND@4; no longer C4.1, C5.1, U$1.GND, U$8.GND
- net N$1: no longer U$1.A5, U$8.A5
- net N$10: now also U1.27; no longer U$1.A1
- net N$11: now also U1.28; no longer U$1.A0
- net N$12: now also U1.7; no longer U$1.10
- net N$14: now also R9.2, U1.9; no longer D2.A, U$1.13
- net N$18: now also U1.50; no longer U$8.8
- net N$19: now also U1.24; no longer U$1.2
- net N$2: now also U1.22; no longer U$1.A4, U$8.A4
- net N$20: now also U1.23; no longer U$1.4
- net N$21: now also U1.29; no longer U$1.8
- net N$22: now also U1.30; no longer U$1.7
- net N$23: now also IC4.4A, U1.46; no longer IC6.I2, U$8.7
- net N$25: now also U1.52; no longer U$8.6
- net N$27: now also U1.53; no longer U$8.5
- net N$28: now also R1.2, U1.12; no longer U$7.2, U$8.A0
- net N$3: now also U1.25; no longer U$1.A3
- net N$30: now also U1.6; no longer U$8.9
- net N$45: now also U$6.3
- net N$46: now also R2.1, U1.31; no longer D1.A, U$8.13
- net N$47: now also R14.2, R16.1, U1.A3; no longer R9.2, U$1.11
- net N$51: now also IC4.4Y, U$6.1, U$6.2; no longer U$6.3
- net N$59: now also U1.49; no longer U$8.A1
- net N$65: now also U1.48; no longer U$8.A2
- net N$71: now also U1.47; no longer U$8.A3
- net N$74: now also JP1.4, U1.36; no longer IC4.4A, U$8.11
- net N$75: now also JP1.5, U1.37; no longer IC4.3A, U$8.10
- net N$8: now also U1.8; no longer U$1.9
- net N$9: now also U1.26; no longer U$1.A2
- net V+: now also R13.1, R13.2, R15.1, U1.A2
Other:
- moved on the sheet: C5, R2, SG1

Commit message: no message
Parts:
- Q1, Q2, Q3, Q4: value IRF540 -> IRFN44Z; device transistor-fet:IRF540 -> transistor-power:PMOSFET_NTO220BH
- R3, R4, R5, R6: value 3k3 -> 33k
Connections:
- net N$2: now also U1.20(SDA); no longer U1.22

Commit message: Z112A case part layout
Parts:
- removed 12V, 12V5, 12V6: Jack 5.5/2.1, SparkFun:POWER_JACKCOMBO
- removed U$10, U$14: DCDC-5V, jolo-lib:DCDC-STEPDOWN
- added 12V-TERM: 12V, SparkFun-Connectors:M025MM
- added 12VIN1, 12VIN2, VREG: Jack 5.5/2.1, SparkFun-Connectors:POWER_JACKPTH
- added R17, R18: 33k, SparkFun:RESISTORPTH1
- added U$1, U$2: MP1584-BUCK, jolo-lib:MP1584-BUCK
- added U$3: ASC712, jolo-lib:ASC712
- 12V1, 12V2, 12V3, 12V4, 5V: device SparkFun:POWER_JACKCOMBO -> SparkFun-Connectors:POWER_JACKPTH
- IC5: device SparkFun:V_REG_78XXSIDE -> SparkFun-PowerIC:V_REG_78XXSINK
- JP1: value (none) -> AUX
- Q1, Q2, Q3, Q4: device transistor-power:PMOSFET_NTO220BH -> transistor-power:IRF540
- X1: value (none) -> STEPPER1
- X2: value (none) -> STEPPER2
Connections:
- net 3.3V renamed N$8
- removed net AGND: 12V.GND, 12V.GNDBREAK, 12V1.GND, 12V1.GNDBREAK, 12V2.GND, 12V2.GNDBREAK, 12V3.GND, 12V3.GNDBREAK, 12V4.GND, 12V4.GNDBREAK, 12V5.GND, 12V5.GNDBREAK, 12V6.GND, 12V6.GNDBREAK, C1.-, C2.2, C3.2, C6.2, C7.2, C9.2, IC1.GND1, IC1.GND2, IC1.GND3, IC1.GND4, IC2.GND1, IC2.GND2, IC2.GND3, IC2.GND4, IC4.GND1, IC4.GND2, IC4.GND3, IC4.GND4, IC5.GND, Q1.S, Q2.S, Q3.S, Q4.S, R3.2, R4.2, R5.2, R6.2, X1.9, X2.9
- removed net DGND: 5V.GND, 5V.GNDBREAK, C10.-, C5.2, C8.-, JP1.10, R15.2, R16.2, SG1.+, TEMP.1, TEMP1.1, TEMP2.1, U$10.GNDIN, U$10.GNDOUT, U$14.GNDIN, U$14.GNDOUT, U$16.1, U$7.1, U1.GND@0, U1.GND@1, U1.GND@2, U1.GND@3, U1.GND@4
- removed net N$79: JP1.9, U1.41
- removed net N$8 (its old number): IC1.3-4EN, U1.8
- new net GND: 12V-TERM.2, 12V1.GND, 12V1.GNDBREAK, 12V2.GND, 12V2.GNDBREAK, 12V3.GND, 12V3.GNDBREAK, 12V4.GND, 12V4.GNDBREAK, 12VIN1.GND, 12VIN1.GNDBREAK, 12VIN2.GND, 12VIN2.GNDBREAK, 5V.GND, 5V.GNDBREAK, C1.-, C10.-, C2.2, C3.2, C5.2, C6.2, C7.2, C8.-, C9.2, IC1.GND1, IC1.GND2, IC1.GND3, IC1.GND4, IC2.GND1, IC2.GND2, IC2.GND3, IC2.GND4, IC4.1A, IC4.2A, IC4.GND1, IC4.GND2, IC4.GND3, IC4.GND4, IC5.GND, IC6.GND, IC6.I6, IC6.I7, JP1.10, Q1.S, Q2.S, Q3.S, Q4.S, R15.2, R16.2, R3.2, R4.2, R5.2, R6.2, SG1.+, TEMP.1, TEMP1.1, TEMP2.1, U$1.GND1, U$1.GND2, U$1.GND3, U$1.GND4, U$16.1, U$2.GND1, U$2.GND2, U$2.GND3, U$2.GND4, U$3.GND, U$7.1, U1.GND@0, U1.GND@1, U1.GND@2, U1.GND@3, U1.GND@4, VREG.GND, VREG.GNDBREAK, X1.9, X2.9
- new net N$17: R1.2, U1.5
- new net N$26: 12V-TERM.1, 12VIN1.PWR, 12VIN2.PWR, C1.+, U$3.Z1
- new net N$48: IC2.3A, U1.A11
- new net N$49: IC2.2A, U1.A12
- new net N$50: IC2.1A, U1.A13
- net +12V: now also U$3.Z2; no longer 12V.PWR, 12V5.PWR, C1.+
- net +5V: now also R17.1, R18.1, U$1.OUT1, U$1.OUT2, U$3.VCC; no longer U$10.VCCOUT
- net N$1: now also R17.2, U1.20(SDA)
- net N$10: now also R9.2, U1.2; no longer IC2.1A, U1.27
- net N$11: now also R8.2, U1.3; no longer IC2.2A, U1.28
- net N$12: now also IC1.1-2EN, IC1.3-4EN, U1.45; no longer U1.7
- net N$14: now also R7.2, U1.4; no longer R9.2, U1.9
- net N$18: now also U1.40; no longer U1.50
- net N$19: now also U1.A8; no longer U1.24
- net N$2: now also R18.2, U1.21(SCL); no longer U1.20(SDA)
- net N$20: now also U1.A9; no longer U1.23
- net N$21: now also IC6.I5, U1.39; no longer IC2.3A, U1.29
- net N$22: now also R13.1, R15.1, U1.A2; no longer IC2.4A, U1.30
- net N$23: now also U1.A4; no longer U1.46
- net N$25: now also U1.42; no longer U1.52
- net N$27: now also U1.43; no longer U1.53
- net N$28: now also F2.2, U$2.IN1, U$2.IN2; no longer R1.2, U1.12
- net N$29: now also U1.41; no longer U1.51
- net N$3: now also U1.A7; no longer U1.25
- net N$30: now also U1.44; no longer U1.6
- net N$31: now also U1.A5; no longer U1.45
- net N$32: now also U$3.OUT, U1.A15; no longer R7.2, U1.11
- net N$33: now also IC2.4A, U1.A10; no longer R8.2, U1.10
- net N$37: now also VREG.PWR; no longer 12V6.PWR
- net N$44: now also U1.A1(TX0)
- net N$46: now also U1.26; no longer U1.31
- net N$53: now also JP1.9; no longer JP1.2
- net N$54: now also IC6.O4; no longer IC6.O5
- net N$55: now also IC6.O3; no longer IC6.O4
- net N$56: now also IC6.O2; no longer IC6.O3
- net N$57: now also IC6.O1; no longer IC6.O2
- net N$59: now also U1.6; no longer U1.49
- net N$63: now also IC6.O5; no longer IC6.O1
- net N$65: now also U1.7; no longer U1.48
- net N$69: now also U$1.IN1, U$1.IN2; no longer U$10.VCCIN
- net N$70: now also JP1.8, U1.33; no longer F2.2, U$14.VCCIN
- net N$71: now also U1.8; no longer U1.47
- net N$72: now also JP1.7, U1.32; no longer JP1.3, U1.35
- net N$74: now also JP1.6, U1.31; no longer JP1.4, U1.36
- net N$75: now also U1.30; no longer U1.37
- net N$76: now also JP1.4, U1.29; no longer JP1.6, U1.38
- net N$77: now also JP1.3, U1.28; no longer JP1.7, U1.39
- net N$78: now also JP1.2, U1.27; no longer JP1.8, U1.40
- net N$9: now also U1.A6; no longer U1.26
- net V+: now also U$2.OUT1, U$2.OUT2; no longer R13.1, R15.1, U$14.VCCOUT, U1.A2
Other:
- moved on the sheet: C1, C2, C5, IC6, JP1, R13, R14, R15, R16, U$16, U1

Commit message: First PCB
Parts:
- removed 12V-TERM: 12V, SparkFun-Connectors:M025MM
- removed C5: 100n, SparkFun:CAPPTH1
- removed J1, J2, J3, J4: POWER_JACKRCA, SparkFun:POWER_JACKRCA
- removed SG1: Buzzer, buzzer2:F/QMBIII
- removed TEMP, TEMP1, TEMP2: Jack 3.5mm, SparkFun:AUDIO-JACKPTH
- removed U$11, U$12, U$13, U$15, U$9: RELAYPTH, SparkFun:RELAYPTH
- removed U$16: I2C, SparkFun:RJ9PTH
- added BUZZER: 5V, SparkFun:CAP_POLPTH4
- added C4: 100uF, SparkFun-Passives:CAP_POLPTH1
- added J5: RJ11, SparkFun-Connectors:RJ11-6PTH
- added JP2: RJ45, SparkFun-Connectors:RJ45-8PTH
- added K1, K2, K3, K4, K5: G5L, relay:G5L
- added X3, X4, X5, X6: TOBU3, con-hirschmann:TOBU3
- JP1: value AUX -> (none); device pinhead:PINHD-1X10 -> SparkFun-Connectors:M05X2PTH
- R10, R11, R12: value 3k3 -> 4k7
- R17, R18: value 33k -> 4k7
Connections:
- removed net N$75: JP1.5, U1.30
- removed net N$76: JP1.4, U1.29
- removed net N$77: JP1.3, U1.28
- removed net N$78: JP1.2, U1.27
- new net N$13: J5.3, U1.17(RX2)
- new net N$79: R1.2, U1.12
- new net N$81: IC2.2A, U1.A13
- new net N$82: IC2.3A, U1.A12
- new net N$83: IC2.4A, U1.A11
- new net N$84: IC2.1A, U1.A10
- net +12V: now also C1.+, C4.+, K11.2, K21.2, K22.P, K31.2, K32.P, K41.2, K42.P, K51.2, K52.P, U1.VIN, X3.1, X4.1, X5.1, X6.1; no longer J1.PWR, J2.PWR, J3.PWR, J4.PWR, U$11.COIL2, U$11.MAIN, U$12.COIL2, U$12.MAIN, U$13.COIL2, U$13.MAIN, U$15.COIL2, U$9.COIL2, U$9.MAIN
- net +5V: now also IC1.VCC1, IC2.VCC1, IC4.VCC1, J5.6, JP1.2, JP2.8; no longer C5.1, IC1.VCC2, IC2.VCC2, IC4.VCC2, JP1.1, TEMP.5, TEMP1.5, TEMP2.5, U$16.4, U1.5V@0, U1.5V@1, U1.5V@2
- net GND: now also BUZZER.-, C4.-, J5.1, JP1.1, JP2.1, JP2.3, JP2.5, JP2.7; no longer 12V-TERM.2, C5.2, JP1.10, SG1.+, TEMP.1, TEMP1.1, TEMP2.1, U$16.1, U1.GND@0, U1.GND@1, U1.GND@2, U1.GND@3
- net N$1: now also J5.4; no longer U$16.2
- net N$10: now also U1.9; no longer U1.2
- net N$11: now also U1.10; no longer U1.3
- net N$14: now also U1.11; no longer U1.4
- net N$15: now also X2.3; no longer X2.1
- net N$16: now also X1.3; no longer X1.1
- net N$17: now also J5.2, U1.16(TX2); no longer R1.2, U1.5
- net N$18: now also IC6.I4; no longer IC6.I1
- net N$19: now also F6.2, K42.S; no longer IC1.2A, U1.A8
- net N$2: now also J5.5; no longer U$16.3
- net N$20: now also F7.2, K52.S; no longer IC1.1A, U1.A9
- net N$23: now also U1.A5; no longer U1.A4
- net N$24: now also BUZZER.+; no longer SG1.-
- net N$25: now also IC6.I2; no longer IC6.I3
- net N$26: no longer 12V-TERM.1, C1.+
- net N$27: now also IC6.I1; no longer IC6.I4
- net N$29: now also IC6.I3; no longer IC6.I2
- net N$3: now also C7.1, IC4.VCC2, IC5.OUT; no longer IC1.3A, U1.A7
- net N$30: now also U1.8; no longer U1.44
- net N$31: now also U1.A4; no longer U1.A5
- net N$33: now also IC1.2A, U1.A9; no longer IC2.4A, U1.A10
- net N$35: now also X3.2; no longer J1.GND, J1.GNDBREAK
- net N$36: now also X4.2; no longer J2.GND, J2.GNDBREAK
- net N$37: now also K12.S; no longer U$15.NO
- net N$38: now also X5.2; no longer J3.GND, J3.GNDBREAK
- net N$4: now also X2.1; no longer X2.3
- net N$45: now also IC4.4Y; no longer IC4.3Y
- net N$46: now also U1.30; no longer U1.26
- net N$48: now also IC1.3A, U1.A8; no longer IC2.3A, U1.A11
- net N$49: now also IC1.4A, U1.A7; no longer IC2.2A, U1.A12
- net N$50: now also IC1.1A, U1.A6; no longer IC2.1A, U1.A13
- net N$51: now also IC4.3Y; no longer IC4.4Y
- net N$53: now also JP1.4, U1.22; no longer JP1.9, U1.34
- net N$54: now also IC6.O3, K41.1; no longer IC6.O4, U$9.COIL1
- net N$55: now also IC6.O4, K51.1; no longer IC6.O3, U$11.COIL1
- net N$56: now also K31.1; no longer U$12.COIL1
- net N$57: now also K21.1; no longer U$13.COIL1
- net N$58: now also IC1.VCC2, IC2.VCC2; no longer IC1.VCC1, IC2.VCC1
- net N$59: now also JP2.6, U1.5; no longer TEMP.2, U1.6
- net N$6: now also X1.1; no longer X1.3
- net N$62: now also JP1.3, U1.23; no longer F7.2, U$13.NO
- net N$63: now also K11.1; no longer U$15.COIL1
- net N$64: now also X6.2; no longer J4.GND, J4.GNDBREAK
- net N$65: now also JP2.4, U1.6; no longer TEMP1.2, U1.7
- net N$66: now also JP1.6, U1.24; no longer F6.2, U$12.NO
- net N$67: now also JP1.5, U1.25; no longer F5.2, U$11.NO
- net N$68: now also JP1.8, U1.26; no longer F4.2, U$9.NO
- net N$70: now also JP1.7, U1.27; no longer JP1.8, U1.33
- net N$71: now also JP2.2, U1.7; no longer TEMP2.2, U1.8
- net N$72: now also JP1.10, U1.28; no longer JP1.7, U1.32
- net N$74: now also JP1.9, U1.29; no longer JP1.6, U1.31
- net N$8: now also F4.2, K22.S; no longer C7.1, IC4.VCC1, IC5.OUT
- net N$9: now also F5.2, K32.S; no longer IC1.4A, U1.A6
- net V+: now also K12.P; no longer U$15.MAIN
Other:
- moved on the sheet: C1, R2
