File: Eagle/focuser.sch (EAGLE design)
At the start: 72 parts, among them IC1 L293D, IC2 L293D, IC4 L293D, IC5 7809, IC6 ULN2003AN, J5 RJ11, K1 G5L, K2 G5L, K3 G5L, K4 G5L, K5 G5L, Q1 IRFN44Z, Q2 IRFN44Z, Q3 IRFN44Z, Q4 IRFN44Z, U1 ARDUINO-MEGAFULL, X1 STEPPER1, X2 STEPPER2, X3 TOBU3, X4 TOBU3, X5 TOBU3, X6 TOBU3

Commit message: PCB fixes
Parts:
- removed JP2: RJ45, SparkFun-Connectors:RJ45-8PTH
- removed U$6: SW motor, SparkFun:RJ9PTH
- removed U$7: Hand control, SparkFun:RJ9PTH
- added C5: 100n, SparkFun:CAPPTH1
- added F8: 6A, SparkFun:PTCPTH
- added U$4, U$5: RJ9, jolo-lib:RJ9
- added U$8: RJ45, jolo-lib:RJ45
- F1, F2, F3: value PTCPTH -> 2A
- F4, F5, F6, F7: value PTCPTH -> 4A
- J5: value RJ11 -> COMM
- JP1: value (none) -> EXT
- X3: value TOBU3 -> PWM1
- X4: value TOBU3 -> PWM2
- X5: value TOBU3 -> PWM3
- X6: value TOBU3 -> PWM4
Connections:
- new net N$75: IC1.1-2EN, IC1.3-4EN, U1.46
- new net N$76: C3.2, C4.+, F8.2, X3.1, X4.1, X5.1, X6.1
- net +12V: now also F8.1, U$3.Z1; no longer C3.1, C4.+, U$3.Z2, X3.1, X4.1, X5.1, X6.1
- net +5V: now also C5.2, U$5.4, U$8.1; no longer JP2.8, U$7.4
- net GND: now also C3.1, C5.1, U$5.1, U$8.2, U$8.4, U$8.6, U$8.8; no longer C3.2, JP2.1, JP2.3, JP2.5, JP2.7, U$7.1
- net N$1: now also R18.2, U1.21(SCL); no longer R17.2, U1.20(SDA)
- net N$12: no longer IC1.1-2EN, IC1.3-4EN
- net N$2: now also R17.2, U1.20(SDA); no longer R18.2, U1.21(SCL)
- net N$26: now also U$3.Z2; no longer U$3.Z1
- net N$34: now also U$5.2; no longer U$7.2
- net N$44: now also U$5.3; no longer U$7.3
- net N$45: now also U$4.3, U$4.4; no longer U$6.3, U$6.4
- net N$51: now also U$4.1, U$4.2; no longer U$6.1, U$6.2
- net N$59: now also U$8.7; no longer JP2.6
- net N$65: now also U$8.5; no longer JP2.4
- net N$71: now also U$8.3; no longer JP2.2
Other:
- moved on the sheet: C3, J5, R17, R18
