File: Eagle/focuser-no-jumper.sch (EAGLE design)
At the start: 36 parts, among them IC1 78xx, U1 L298

Commit message: Arduino / Eagle updates
Parts:
- removed .: JUMPER-3PTH, SparkFun:JUMPER-3PTH
- removed ...: (no value), SparkFun:JUMPER-2PTH
- added ..1, ..2: JUMPER-3PTH, SparkFun:JUMPER-3PTH
- D1, D2: device SparkFun:DIODEPTH -> diode:1N4004
- SG1: device buzzer:F/QMBIII -> buzzer2:F/QMBIII
- renumbered 0.9A to 1A
Connections:
- removed net N$24 (its old number): CONTROL.1, MANUAL.5, NANO.D3
- removed net N$3: NANO.A0, U1.ENA, U1.ENB
- removed net N$36: NANO.A7, R5.1
- removed net VCC: 12V.GND, PWR.1
- new net N$2: CONTROL.1, MANUAL.5, NANO.D7
- new net N$30: 12V.PWR, PWR.1
- new net N$31: ..1.1, NANO.D10
- new net N$42: NANO.D11, U1.ENA, U1.ENB
- new net N$43: ..1.3, NANO.A1
- net +5: now also ...2; no longer ....2
- net GND: now also ...1, 12V.GND, 12V.GNDBREAK; no longer ..1, 12V.PWR
- net N$12: now also NANO.A0, R5.1; no longer ..3, NANO.A5
- net N$13: now also NANO.A5; no longer NANO.A1
- net N$15: now also NANO.A4; no longer NANO.A2
- net N$18: now also ..1.2, NANO.D9; no longer CONTROL.2, MANUAL.2, NANO.D4
- net N$25: now also ...3, NANO.D12; no longer ..2, NANO.A6
- net N$32: now also ..2.3, NANO.D3; no longer ...3, NANO.D8
- net N$33: now also NANO.D4, R2.1; no longer ...2, NANO.D9
- net N$34: now also ..2.2, NANO.D5; no longer ...1, NANO.D10
- net N$35: now also ..2.1, NANO.D6; no longer NANO.D5, R2.1
- net N$4: now also NANO.A2; no longer NANO.A4
- net N$8: now also CONTROL.2, MANUAL.2, NANO.D8; no longer ....1, NANO.D7
Other:
- moved on the sheet: .., C5, CONTROL, LED, MANUAL, R2, R3, R5, RJ45, SG1
