File: Eagle/focuser.brd (EAGLE design)
At the start: 54.6 x 116.2 mm, 18 parts, among them IC1 L293D, IC2 L293D, IC3 PCF8574P

Commit message: Work continues... VB script update
Connections:
- new net N$10: U$1.6
- new net N$11: U$1.5
- new net N$12: U$1.3
- new net N$13: U$1.11
- new net N$14: U$1.13
- new net N$3: U$1.A3, U$7.STEP
- new net N$4: U$1.A2, U$7.DIR
- new net N$5: U$1.A1, U$6.STEP
- new net N$6: U$1.A0, U$6.DIR
- new net N$7: U$1.10, U$7.EN
- new net N$8: U$1.9, U$6.EN
Changed lines of the file:
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@@
 </signal>
 <signal name="N$1">
-<contactref element="U$8" pad="A5"/>
 <contactref element="U$1" pad="A5"/>
 <contactref element="IC3" pad="14"/>
+<contactref element="U$8" pad="A5"/>
 <wire x1="-56.515" y1="20.955" x2="-60.325" y2="-29.845" width="0" layer="19" extent="1-1"/>
 <wire x1="-6.35" y1="20.955" x2="-56.515" y2="20.955" width="0" layer="19" extent="1-1"/>
 </signal>
 <signal name="N$2">
-<contactref element="U$8" pad="A4"/>
 <contactref element="U$1" pad="A4"/>
 <contactref element="IC3" pad="15"/>
+<contactref element="U$8" pad="A4"/>
 <wire x1="-56.515" y1="18.415" x2="-62.865" y2="-29.845" width="0" layer="19" extent="1-1"/>
 <wire x1="-6.35" y1="18.415" x2="-56.515" y2="18.415" width="0" layer="19" extent="1-1"/>
@@
 <contactref element="IC3" pad="8"/>
 </signal>
+<signal name="N$3">
+<contactref element="U$1" pad="A3"/>
+<contactref element="U$7" pad="STEP"/>
+<wire x1="-3.175" y1="19.685" x2="-50.165" y2="1.27" width="0" layer="19" extent="1-1"/>
+</signal>
+<signal name="N$4">
+<contactref element="U$1" pad="A2"/>
+<contactref element="U$7" pad="DIR"/>
+<wire x1="-3.175" y1="17.145" x2="-50.165" y2="-1.27" width="0" layer="19" extent="1-1"/>
+</signal>
+<signal name="N$5">
+<contactref element="U$1" pad="A1"/>
+<contactref element="U$6" pad="STEP"/>
+<wire x1="-3.175" y1="14.605" x2="-34.29" y2="1.27" width="0" layer="19" extent="1-1"/>
+</signal>
+<signal name="N$6">
+<contactref element="U$1" pad="A0"/>
+<contactref element="U$6" pad="DIR"/>
+<wire x1="-3.175" y1="12.065" x2="-34.29" y2="-1.27" width="0" layer="19" extent="1-1"/>
+</signal>
+<signal name="N$7">
+<contactref element="U$1" pad="10"/>
+<contactref element="U$7" pad="EN"/>
+<wire x1="-3.175" y1="1.905" x2="-50.165" y2="16.51" width="0" layer="19" extent="1-1"/>
+</signal>
+<signal name="N$8">
+<contactref element="U$1" pad="9"/>
+<contactref element="U$6" pad="EN"/>
+<wire x1="-34.29" y1="16.51" x2="-18.415" y2="1.905" width="0" layer="19" extent="1-1"/>
+</signal>
+<signal name="N$10">
+<contactref element="U$1" pad="6"/>
+</signal>
+<signal name="N$11">
+<contactref element="U$1" pad="5"/>
+</signal>
+<signal name="N$12">
+<contactref element="U$1" pad="3"/>
+</signal>
+<signal name="N$13">
+<contactref element="U$1" pad="11"/>
+</signal>
+<signal name="N$14">
+<contactref element="U$1" pad="13"/>
+</signal>
 </signals>

Commit message: Schematic update
Parts:
- removed .., ..1, ..2: (no value), SparkFun:1X03
- removed IC3: PCF8574P, micro-philips:DIL16
- added 12V1, 12V2, 12V3, 12V4, 12V5, 12V6: Jack 5.5/2.1, SparkFun:POWER_JACK_COMBO
- added C1: 1000u, SparkFun:CPOL-RADIAL-1000UF-25V
- added C10, C8: 10u, SparkFun:CPOL-RADIAL-10UF-25V
- added C2, C3, C4, C5, C6, C7, C9: 100n, SparkFun:CAP-PTH-5MM
- added D1, D2: (no value), SparkFun:DIODE-1N4148
- added F1, F2, F3, F4, F5, F6, F7: PTCPTH, SparkFun:PTC
- added IC4: L293D, st-microelectronics:DIL16
- added IC5: 7809, SparkFun:TO220-IGO
- added IC6: ULN2003AN, uln-udn:DIL16
- added J1, J2, J3, J4: POWER_JACKRCA, SparkFun:RCA
- added Q1, Q2, Q3, Q4: IRF540, transistor-fet:TO220
- added R1, R7, R8, R9: 100, SparkFun:AXIAL-0.3
- added R10, R11, R12, R3, R4, R5, R6: 3k3, SparkFun:AXIAL-0.3
- added TEMP1, TEMP2: Jack 3.5mm, SparkFun:AUDIO-JACK
- added U$10, U$14: DCDC-5V, jolo-lib:DCDC-STEPDOWN
- added U$11, U$12, U$13, U$15, U$9: RELAYPTH, SparkFun:RELAY-G5Q
- added U$16: I2C, SparkFun:RJ9
- added X1, X2: (no value), SparkFun:DB9
- U$6: value A4988-MODULE -> SW motor; device jolo-lib:A4988-MODULE -> SparkFun:RJ9
- U$7: value A4988-MODULE -> Hand control; device jolo-lib:A4988-MODULE -> SparkFun:RJ9
- moved U$6 482.9 mm to (-238.8, -421.0)
- moved U$7 481.3 mm to (-250.8, -421.0)
- moved IC1 402.0 mm to (-219.7, -376.6)
- moved IC2 402.0 mm to (-219.7, -388.6)
Connections:
- removed net GMOT: U$6.GMOT, U$7.GMOT
- removed net GND1: IC1.4, IC2.4
- removed net GND3: IC1.13, IC2.13
- removed net GND4: IC1.12, IC2.12
- removed net VCC1: IC1.16, IC2.16
- removed net VCC2: IC1.8, IC2.8, U$1.VCC2, U$8.VCC2
- removed net VDD: IC3.16, U$6.VDD, U$7.VDD
- removed net VMOT: U$6.VMOT, U$7.VMOT
- removed net VSS: IC3.8
- new net +12V: 12V.POWER, 12V5.POWER, C1.1, C2.1, C3.1, C9.1, F1.P$1, F2.P$1, F3.P$2, IC5.IN, IC6.9, J1.BREAK, J2.BREAK, J3.BREAK, J4.BREAK, U$11.1, U$11.2, U$12.1, U$12.2, U$13.1, U$13.2, U$15.1, U$9.1, U$9.2
- new net +5V: C10.1, C4.2, C5.2, C8.1, IC1.8, IC2.8, IC4.8, R10.P$2, R11.P$2, R12.P$2, TEMP.5, TEMP1.5, TEMP2.5, U$1.VCC2, U$10.VCCOUT, U$16.4, U$7.4, U$8.VCC2
- new net 3.3V: C7.1, IC4.16, IC5.OUT
- new net AGND: 12V.GND, 12V.GND@1, 12V1.GND, 12V1.GND@1, 12V2.GND, 12V2.GND@1, 12V3.GND, 12V3.GND@1, 12V4.GND, 12V4.GND@1, 12V5.GND, 12V5.GND@1, 12V6.GND, 12V6.GND@1, C1.2, C2.2, C3.2, C6.2, C7.2, C9.2, IC1.12, IC1.13, IC1.4, IC1.5, IC2.12, IC2.13, IC2.4, IC2.5, IC4.12, IC4.13, IC4.4, IC4.5, IC5.GND, Q1.3, Q2.3, Q3.3, Q4.3, R3.P$2, R4.P$2, R5.P$2, R6.P$2, X1.9, X2.9
- new net DGND: C10.2, C4.1, C5.1, C8.2, SG1.-, TEMP.1, TEMP1.1, TEMP2.1, U$1.GND, U$10.GNDIN, U$10.GNDOUT, U$14.GNDIN, U$14.GNDOUT, U$16.1, U$7.1, U$8.GND
- new net N$15: IC2.6, X2.1
- new net N$16: IC1.6, X1.1
- new net N$17: D1.C, D2.C, R2.P$1
- new net N$18: IC6.1, U$8.8
- new net N$19: IC1.7, U$1.2
- new net N$20: IC1.2, U$1.4
- new net N$21: IC2.10, U$1.8
- new net N$22: IC2.15, U$1.7
- new net N$23: IC6.2, U$8.7
- new net N$25: IC6.3, U$8.6
- new net N$27: IC6.4, U$8.5
- new net N$28: U$7.2, U$8.A0
- new net N$30: IC4.1, IC4.9, U$8.9
- new net N$35: J1.BARREL, J1.SPRING, Q1.2
- new net N$36: J2.BARREL, J2.SPRING, Q2.2
- new net N$37: 12V6.POWER, U$15.3
- new net N$38: J3.BARREL, J3.SPRING, Q3.2
- new net N$39: Q4.1, R6.P$1, R9.P$1
- new net N$40: Q3.1, R5.P$1, R8.P$1
- new net N$41: Q2.1, R4.P$1, R7.P$1
- new net N$42: Q1.1, R1.P$1, R3.P$1
- new net N$43: 12V1.POWER, F4.P$1
- new net N$45: IC4.11, U$6.4
- new net N$46: D1.A, U$8.13
- new net N$47: R9.P$2, U$1.11
- new net N$48: R8.P$2, U$1.3
- new net N$49: R7.P$2, U$1.5
- new net N$50: R1.P$2, U$1.6
- new net N$51: U$6.3
- new net N$52: 12V2.POWER, F5.P$1
- new net N$54: IC6.12, U$9.5
- new net N$55: IC6.13, U$11.5
- new net N$56: IC6.14, U$12.5
- new net N$57: IC6.15, U$13.5
- new net N$58: C6.1, F3.P$1, IC1.16, IC2.16, X1.5, X2.5
- new net N$59: R12.P$1, TEMP.2, U$8.A1
- new net N$60: 12V3.POWER, F6.P$1
- new net N$61: 12V4.POWER, F7.P$1
- new net N$62: F7.P$2, U$13.3
- new net N$63: IC6.16, U$15.5
- new net N$64: J4.BARREL, J4.SPRING, Q4.2
- new net N$65: R11.P$1, TEMP1.2, U$8.A2
- new net N$66: F6.P$2, U$12.3
- new net N$67: F5.P$2, U$11.3
- new net N$68: F4.P$2, U$9.3
- new net N$69: F1.P$2, U$10.VCCIN
- new net N$70: F2.P$2, U$14.VCCIN
- new net N$71: R10.P$1, TEMP2.2, U$8.A3
- new net N$73: IC2.11, X2.4
- new net N$74: IC4.15, U$8.11
- new net N$75: IC4.10, U$8.10
- new net N$9: IC1.15, U$1.A2
- new net V+: U$14.VCCOUT, U$15.2
- net GND: now also IC6.8; no longer SG1.-, U$1.GND, U$6.GND, U$7.GND, U$8.GND
- net GND2: no longer IC1.5, IC2.5
- net N$1: now also U$16.2; no longer IC3.14
- net N$10: now also IC2.2, U$1.A1; no longer U$1.6
- net N$11: now also IC2.7, U$1.A0; no longer U$1.5
- net N$12: now also IC2.1, IC2.9, U$1.10; no longer U$1.3
- net N$13: now also IC2.3, X2.2; no longer U$1.11
- net N$14: now also D2.A
- net N$2: now also U$16.3; no longer IC3.15
- net N$3: now also IC1.10; no longer U$7.STEP
- net N$4: now also IC2.14, X2.3; no longer U$1.A2, U$7.DIR
- net N$5: now also IC1.3, X1.2; no longer U$1.A1, U$6.STEP
- net N$6: now also IC1.14, X1.3; no longer U$1.A0, U$6.DIR
- net N$7: now also IC1.11, X1.4; no longer U$1.10, U$7.EN
- net N$8: now also IC1.9; no longer U$6.EN
Routing:
- net DGND: track 0.00 -> 11.3 mm
- net GND: track 38.7 -> 27.4 mm

Commit message: no message
Parts:
- removed C4: 100n, SparkFun:CAP-PTH-5MM
- removed D1, D2: (no value), SparkFun:DIODE-1N4148
- removed U$1, U$8: ARDUINO-MINI-PRO, jolo-lib:ARDUINO-MINI-PRO
- removed U$2, U$3, U$4, U$5: (no value), holes:3,6
- added 5V: Jack 5.5/2.1, SparkFun:POWER_JACK_COMBO
- added JP1: (no value), pinhead:1X10
- added R13, R14: 2k, SparkFun:AXIAL-0.3
- added R15, R16: 1k, SparkFun:AXIAL-0.3
- added U1: ARDUINO-MEGAFULL, SparkFun-Boards:ARDUINO_MEGA
- IC5: device SparkFun:TO220-IGO -> SparkFun:78XXL
- moved U$6 357.5 mm to (-121.9, -83.2), turned to 180 degrees
- moved C9 345.6 mm to (-124.5, -100.3), turned to 270 degrees
- moved C7 340.4 mm to (-127.6, -100.3), turned to 90 degrees
- moved IC5 340.1 mm to (-135.9, -88.3), turned to 180 degrees
- moved C10 339.1 mm to (-51.4, -169.5), turned to 90 degrees
- moved 12V6 335.4 mm to (36.2, -79.4), turned to 270 degrees
- moved IC2 328.3 mm to (-60.3, -101.6)
- moved IC4 324.5 mm to (-111.8, -101.0)
- moved F5 320.2 mm to (6.99, -92.7), turned to 180 degrees
- moved U$16 316.2 mm to (-61.6, -177.2)
- moved TEMP 315.8 mm to (-90.4, -180.0), turned to 90 degrees
- moved C1 315.3 mm to (38.1, -150.5), turned to 270 degrees
- moved C2 313.8 mm to (38.7, -164.5), turned to 270 degrees
- moved F1 313.7 mm to (38.7, -129.5), turned to 270 degrees
- moved F2 310.2 mm to (32.4, -129.5), turned to 90 degrees
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Connections:
- removed net GND2: U$1.GND2, U$8.GND2
- removed net GRN: U$1.GRN, U$8.GRN
- removed net N$17: D1.C, D2.C, R2.P$1
- removed net N$48: R8.P$2, U$1.3
- removed net N$49: R7.P$2, U$1.5
- removed net N$50: R1.P$2, U$1.6
- removed net RAW: U$1.RAW, U$8.RAW
- removed net VCC: U$1.VCC, U$8.VCC
- new net N$29: IC6.2, U1.51
- new net N$31: IC4.10, U1.45
- new net N$32: R7.P$2, U1.11
- new net N$33: R8.P$2, U1.10
- new net N$34: U$7.2, U1.A0
- new net N$44: U$7.3
- new net N$53: JP1.2, U1.34
- new net N$72: JP1.3, U1.35
- new net N$76: JP1.6, U1.38
- new net N$77: JP1.7, U1.39
- new net N$78: JP1.8, U1.40
- new net N$79: JP1.9, U1.41
- net +12V: now also R14.P$1
- net +5V: now also 5V.POWER, C5.1, JP1.1, U1.5V@0, U1.5V@1, U1.5V@2; no longer C4.2, C5.2, U$1.VCC2, U$8.VCC2
- net DGND: now also 5V.GND, 5V.GND@1, C5.2, JP1.10, R15.P$2, R16.P$2, U1.GND@0, U1.GND@1, U1.GND@2, U1.GND@3, U1.GND@4; no longer C4.1, C5.1, U$1.GND, U$8.GND
- net N$1: no longer U$1.A5, U$8.A5
- net N$10: now also U1.27; no longer U$1.A1
- net N$11: now also U1.28; no longer U$1.A0
- net N$12: now also U1.7; no longer U$1.10
- net N$14: now also R9.P$2, U1.9; no longer D2.A, U$1.13
- net N$18: now also U1.50; no longer U$8.8
- net N$19: now also U1.24; no longer U$1.2
- net N$2: now also U1.22; no longer U$1.A4, U$8.A4
- net N$20: now also U1.23; no longer U$1.4
- net N$21: now also U1.29; no longer U$1.8
- net N$22: now also U1.30; no longer U$1.7
- net N$23: now also IC4.15, U1.46; no longer IC6.2, U$8.7
- net N$25: now also U1.52; no longer U$8.6
- net N$27: now also U1.53; no longer U$8.5
- net N$28: now also R1.P$2, U1.12; no longer U$7.2, U$8.A0
- net N$3: now also U1.25; no longer U$1.A3
- net N$30: now also U1.6; no longer U$8.9
- net N$45: now also U$6.3
- net N$46: now also R2.P$1, U1.31; no longer D1.A, U$8.13
- net N$47: now also R14.P$2, R16.P$1, U1.A3; no longer R9.P$2, U$1.11
- net N$51: now also IC4.14, U$6.1, U$6.2; no longer U$6.3
- net N$59: now also U1.49; no longer U$8.A1
- net N$65: now also U1.48; no longer U$8.A2
- net N$71: now also U1.47; no longer U$8.A3
- net N$74: now also JP1.4, U1.36; no longer IC4.15, U$8.11
- net N$75: now also JP1.5, U1.37; no longer IC4.10, U$8.10
- net N$8: now also U1.8; no longer U$1.9
- net N$9: now also U1.26; no longer U$1.A2
- net V+: now also R13.P$1, R13.P$2, R15.P$1, U1.A2
Routing:
- net GND: track 27.4 -> 0.00 mm
- net DGND: track 11.3 -> 0.00 mm
- net N$24: track 8.15 -> 0.00 mm
- removed copper zone on layer 16, net GND
Other:
- board outline removed
- board text removed: "+"
- board text removed: "+5"
- board text removed: "-"
- board text removed: "0"
- board text removed: "2014-04"
- board text removed: "A2"
- board text removed: "ASCOM JoloFocuser"
- board text removed: "C"
- board text removed: "D10"
- board text removed: "D13"
- board text removed: "D3"
- board text removed: "D5"
- board text removed: "D6"
- board text removed: "D9"
- board text removed: "E"
- board text removed: "GND"
- board text removed: "Polymer Fuse"
- board text removed: "rev. 2.0"

Commit message: no message
Parts:
- Q1, Q2, Q3, Q4: value IRF540 -> IRFN44Z; device transistor-fet:TO220 -> transistor-power:TO220BH
- R3, R4, R5, R6: value 3k3 -> 33k
- moved Q4 200.3 mm to (-179.1, -184.2), turned to 0 degrees
- moved Q3 152.2 mm to (-167.0, -184.2), turned to 0 degrees
- moved Q2 144.1 mm to (-154.9, -184.2), turned to 0 degrees
Connections:
- net AGND: now also Q1.S, Q2.S, Q3.S, Q4.S; no longer Q1.3, Q2.3, Q3.3, Q4.3
- net N$2: now also U1.20; no longer U1.22
- net N$35: now also Q1.D; no longer Q1.2
- net N$36: now also Q2.D; no longer Q2.2
- net N$38: now also Q3.D; no longer Q3.2
- net N$39: now also Q4.G; no longer Q4.1
- net N$40: now also Q3.G; no longer Q3.1
- net N$41: now also Q2.G; no longer Q2.1
- net N$42: now also Q1.G; no longer Q1.1
- net N$64: now also Q4.D; no longer Q4.2

Commit message: Z112A case part layout
Parts:
- removed 12V, 12V5, 12V6: Jack 5.5/2.1, SparkFun:POWER_JACK_COMBO
- removed U$10, U$14: DCDC-5V, jolo-lib:DCDC-STEPDOWN
- added 12V-TERM: 12V, SparkFun-Connectors:SCREWTERMINAL-5MM-2
- added 12VIN1, 12VIN2, VREG: Jack 5.5/2.1, SparkFun-Connectors:POWER_JACK_PTH
- added R17, R18: 33k, SparkFun:AXIAL-0.3
- added U$1, U$2: MP1584-BUCK, jolo-lib:DCDC-1584
- added U$3: ASC712, jolo-lib:ASC712
- 12V1, 12V2, 12V3, 12V4, 5V: device SparkFun:POWER_JACK_COMBO -> SparkFun-Connectors:POWER_JACK_PTH
- IC5: device SparkFun:78XXL -> SparkFun-PowerIC:TO220-IGO
- JP1: value (none) -> AUX
- Q1, Q2, Q3, Q4: device transistor-power:TO220BH -> transistor-power:TO220BV
- X1: value (none) -> STEPPER1
- X2: value (none) -> STEPPER2
- moved Q3 423.7 mm to (143.5, 104.1), turned to 180 degrees
- moved Q2 405.9 mm to (130.8, 104.1), turned to 180 degrees
- moved Q4 399.7 mm to (97.8, 104.1), turned to 180 degrees
- moved J2 342.6 mm to (128.3, 119.4), turned to 270 degrees
- moved J3 341.7 mm to (141.0, 119.4), turned to 270 degrees
- moved J4 319.4 mm to (102.9, 119.4), turned to 270 degrees
- moved J1 318.9 mm to (115.6, 119.4), turned to 270 degrees
- moved C3 305.3 mm to (108.0, 97.8)
- moved R8 300.3 mm to (143.5, 95.2)
- moved R4 290.4 mm to (130.8, 99.1), turned to 180 degrees
- moved R5 288.8 mm to (97.8, 99.1), turned to 180 degrees
- moved Q1 284.4 mm to (118.1, 104.1), turned to 180 degrees
- moved R7 280.0 mm to (130.8, 95.2)
- moved R3 275.7 mm to (118.1, 99.1), turned to 180 degrees
- moved C8 271.3 mm to (68.6, 16.5), turned to 180 degrees
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Connections:
- net 3.3V renamed N$8
- removed net AGND: 12V.GND, 12V.GND@1, 12V1.GND, 12V1.GND@1, 12V2.GND, 12V2.GND@1, 12V3.GND, 12V3.GND@1, 12V4.GND, 12V4.GND@1, 12V5.GND, 12V5.GND@1, 12V6.GND, 12V6.GND@1, C1.2, C2.2, C3.2, C6.2, C7.2, C9.2, IC1.12, IC1.13, IC1.4, IC1.5, IC2.12, IC2.13, IC2.4, IC2.5, IC4.12, IC4.13, IC4.4, IC4.5, IC5.GND, Q1.S, Q2.S, Q3.S, Q4.S, R3.P$2, R4.P$2, R5.P$2, R6.P$2, X1.9, X2.9
- removed net DGND: 5V.GND, 5V.GND@1, C10.2, C5.2, C8.2, JP1.10, R15.P$2, R16.P$2, SG1.-, TEMP.1, TEMP1.1, TEMP2.1, U$10.GNDIN, U$10.GNDOUT, U$14.GNDIN, U$14.GNDOUT, U$16.1, U$7.1, U1.GND@0, U1.GND@1, U1.GND@2, U1.GND@3, U1.GND@4
- removed net N$79: JP1.9, U1.41
- removed net N$8 (its old number): IC1.9, U1.8
- new net N$17: R1.P$2, U1.5
- new net N$26: 12V-TERM.1, 12VIN1.PWR, 12VIN2.PWR, C1.1, U$3.Z1
- new net N$48: IC2.10, U1.A11
- new net N$49: IC2.7, U1.A12
- new net N$50: IC2.2, U1.A13
- net +12V: now also U$3.Z2; no longer 12V.POWER, 12V5.POWER, C1.1
- net +5V: now also 5V.PWR, R17.P$1, R18.P$1, U$1.OUT1, U$1.OUT2, U$3.VCC; no longer 5V.POWER, U$10.VCCOUT
- net GND: now also 12V-TERM.2, 12V1.GND, 12V1.GNDBREAK, 12V2.GND, 12V2.GNDBREAK, 12V3.GND, 12V3.GNDBREAK, 12V4.GND, 12V4.GNDBREAK, 12VIN1.GND, 12VIN1.GNDBREAK, 12VIN2.GND, 12VIN2.GNDBREAK, 5V.GND, 5V.GNDBREAK, C1.2, C10.2, C2.2, C3.2, C5.2, C6.2, C7.2, C8.2, C9.2, IC1.12, IC1.13, IC1.4, IC1.5, IC2.12, IC2.13, IC2.4, IC2.5, IC4.12, IC4.13, IC4.2, IC4.4, IC4.5, IC4.7, IC5.GND, IC6.6, IC6.7, JP1.10, Q1.S, Q2.S, Q3.S, Q4.S, R15.P$2, R16.P$2, R3.P$2, R4.P$2, R5.P$2, R6.P$2, SG1.-, TEMP.1, TEMP1.1, TEMP2.1, U$1.GND1, U$1.GND2, U$1.GND3, U$1.GND4, U$16.1, U$2.GND1, U$2.GND2, U$2.GND3, U$2.GND4, U$3.GND, U$7.1, U1.GND@0, U1.GND@1, U1.GND@2, U1.GND@3, U1.GND@4, VREG.GND, VREG.GNDBREAK, X1.9, X2.9
- net N$1: now also R17.P$2, U1.20
- net N$10: now also R9.P$2, U1.2; no longer IC2.2, U1.27
- net N$11: now also R8.P$2, U1.3; no longer IC2.7, U1.28
- net N$12: now also IC1.1, IC1.9, U1.45; no longer U1.7
- net N$14: now also R7.P$2, U1.4; no longer R9.P$2, U1.9
- net N$18: now also U1.40; no longer U1.50
- net N$19: now also U1.A8; no longer U1.24
- net N$2: now also R18.P$2, U1.21; no longer U1.20
- net N$20: now also U1.A9; no longer U1.23
- net N$21: now also IC6.5, U1.39; no longer IC2.10, U1.29
- net N$22: now also R13.P$1, R15.P$1, U1.A2; no longer IC2.15, U1.30
- net N$23: now also U1.A4; no longer U1.46
- net N$25: now also U1.42; no longer U1.52
- net N$27: now also U1.43; no longer U1.53
- net N$28: now also F2.P$2, U$2.IN1, U$2.IN2; no longer R1.P$2, U1.12
- net N$29: now also U1.41; no longer U1.51
- net N$3: now also U1.A7; no longer U1.25
- net N$30: now also U1.44; no longer U1.6
- net N$31: now also U1.A5; no longer U1.45
- net N$32: now also U$3.OUT, U1.A15; no longer R7.P$2, U1.11
- net N$33: now also IC2.15, U1.A10; no longer R8.P$2, U1.10
- net N$37: now also VREG.PWR; no longer 12V6.POWER
- net N$43: now also 12V1.PWR; no longer 12V1.POWER
- net N$44: now also U1.A1
- net N$46: now also U1.26; no longer U1.31
- net N$52: now also 12V2.PWR; no longer 12V2.POWER
- net N$53: now also JP1.9; no longer JP1.2
- net N$54: now also IC6.13; no longer IC6.12
- net N$55: now also IC6.14; no longer IC6.13
- net N$56: now also IC6.15; no longer IC6.14
- net N$57: now also IC6.16; no longer IC6.15
- net N$59: now also U1.6; no longer U1.49
- net N$60: now also 12V3.PWR; no longer 12V3.POWER
- net N$61: now also 12V4.PWR; no longer 12V4.POWER
- net N$63: now also IC6.12; no longer IC6.16
- net N$65: now also U1.7; no longer U1.48
- net N$69: now also U$1.IN1, U$1.IN2; no longer U$10.VCCIN
- net N$70: now also JP1.8, U1.33; no longer F2.P$2, U$14.VCCIN
- net N$71: now also U1.8; no longer U1.47
- net N$72: now also JP1.7, U1.32; no longer JP1.3, U1.35
- net N$74: now also JP1.6, U1.31; no longer JP1.4, U1.36
- net N$75: now also U1.30; no longer U1.37
- net N$76: now also JP1.4, U1.29; no longer JP1.6, U1.38
- net N$77: now also JP1.3, U1.28; no longer JP1.7, U1.39
- net N$78: now also JP1.2, U1.27; no longer JP1.8, U1.40
- net N$9: now also U1.A6; no longer U1.26
- net V+: now also U$2.OUT1, U$2.OUT2; no longer R13.P$1, R15.P$1, U$14.VCCOUT, U1.A2
Other:
- board outline added: 191.8 x 149.9 mm
