File: Eagle/focuser.brd (EAGLE design)
At the start: 191.8 x 149.9 mm, 75 parts, among them IC1 L293D, IC2 L293D, IC4 L293D, IC5 7809, IC6 ULN2003AN, J1 POWER_JACKRCA, J2 POWER_JACKRCA, J3 POWER_JACKRCA, J4 POWER_JACKRCA, Q1 IRFN44Z, Q2 IRFN44Z, Q3 IRFN44Z, Q4 IRFN44Z, U1 ARDUINO-MEGAFULL, X1 STEPPER1, X2 STEPPER2

Commit message: First PCB
Parts:
- removed 12V-TERM: 12V, SparkFun-Connectors:SCREWTERMINAL-5MM-2
- removed C5: 100n, SparkFun:CAP-PTH-5MM
- removed J1, J2, J3, J4: POWER_JACKRCA, SparkFun:RCA
- removed SG1: Buzzer, buzzer2:F/QMBIII
- removed TEMP, TEMP1, TEMP2: Jack 3.5mm, SparkFun:AUDIO-JACK
- removed U$11, U$12, U$13, U$15, U$9: RELAYPTH, SparkFun:RELAY-G5Q
- removed U$16: I2C, SparkFun:RJ9
- added BUZZER: 5V, SparkFun:CPOL-RADIAL-1000UF-25V
- added C4: 100uF, SparkFun-Passives:CPOL-RADIAL-100UF-25V
- added J5: RJ11, SparkFun-Connectors:RJ11-6
- added JP2: RJ45, SparkFun-Connectors:RJ45-8
- added K1, K2, K3, K4, K5: G5L, relay:G5LE
- added X3, X4, X5, X6: TOBU3, con-hirschmann:TOBU3
- JP1: value AUX -> (none); device pinhead:1X10 -> SparkFun-Connectors:AVR_ICSP
- R10, R11, R12: value 3k3 -> 4k7
- R17, R18: value 33k -> 4k7
- moved VREG 114.7 mm to (115.6, -5.08), turned to 0 degrees
- moved 12V1 102.9 mm to (171.4, 97.8), turned to 90 degrees
- moved R6 102.4 mm to (47.0, 64.8), turned to 270 degrees
- moved R8 98.8 mm to (54.6, 52.1), turned to 270 degrees
- moved 5V 97.4 mm to (129.5, -5.08), turned to 0 degrees
- moved 12V4 95.6 mm to (171.4, 59.7), turned to 90 degrees
- moved 12V2 94.9 mm to (171.4, 85.1), turned to 90 degrees
- moved 12V3 90.9 mm to (171.4, 72.4), turned to 90 degrees
- moved R7 90.9 mm to (50.8, 52.1), turned to 270 degrees
- moved R4 83.6 mm to (54.6, 64.8), turned to 270 degrees
- moved R1 83.2 mm to (47.0, 52.1), turned to 270 degrees
- moved R3 75.5 mm to (50.8, 64.8), turned to 270 degrees
- moved F5 73.8 mm to (138.4, 90.2)
- moved F4 73.7 mm to (148.6, 90.2)
- moved C1 67.8 mm to (143.5, 6.35), turned to 90 degrees
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Connections:
- removed net N$75: JP1.5, U1.30
- removed net N$76: JP1.4, U1.29
- removed net N$77: JP1.3, U1.28
- removed net N$78: JP1.2, U1.27
- new net N$13: J5.3, U1.17
- new net N$79: R1.P$2, U1.12
- new net N$81: IC2.7, U1.A13
- new net N$82: IC2.10, U1.A12
- new net N$83: IC2.15, U1.A11
- new net N$84: IC2.2, U1.A10
- net +12V: now also C1.1, C4.1, K1.2, K2.2, K2.P, K3.2, K3.P, K4.2, K4.P, K5.2, K5.P, U1.VIN, X3.1, X4.1, X5.1, X6.1; no longer J1.BREAK, J2.BREAK, J3.BREAK, J4.BREAK, U$11.1, U$11.2, U$12.1, U$12.2, U$13.1, U$13.2, U$15.1, U$9.1, U$9.2
- net +5V: now also IC1.16, IC2.16, IC4.16, J5.6, JP1.2, JP2.8; no longer C5.1, IC1.8, IC2.8, IC4.8, JP1.1, TEMP.5, TEMP1.5, TEMP2.5, U$16.4, U1.5V@0, U1.5V@1, U1.5V@2
- net GND: now also BUZZER.2, C4.2, J5.1, JP1.1, JP2.1, JP2.3, JP2.5, JP2.7; no longer 12V-TERM.2, C5.2, JP1.10, SG1.-, TEMP.1, TEMP1.1, TEMP2.1, U$16.1, U1.GND@0, U1.GND@1, U1.GND@2, U1.GND@3
- net N$1: now also J5.4; no longer U$16.2
- net N$10: now also U1.9; no longer U1.2
- net N$11: now also U1.10; no longer U1.3
- net N$14: now also U1.11; no longer U1.4
- net N$15: now also X2.3; no longer X2.1
- net N$16: now also X1.3; no longer X1.1
- net N$17: now also J5.2, U1.16; no longer R1.P$2, U1.5
- net N$18: now also IC6.4; no longer IC6.1
- net N$19: now also F6.P$2, K4.S; no longer IC1.7, U1.A8
- net N$2: now also J5.5; no longer U$16.3
- net N$20: now also F7.P$2, K5.S; no longer IC1.2, U1.A9
- net N$23: now also U1.A5; no longer U1.A4
- net N$24: now also BUZZER.1; no longer SG1.+
- net N$25: now also IC6.2; no longer IC6.3
- net N$26: no longer 12V-TERM.1, C1.1
- net N$27: now also IC6.1; no longer IC6.4
- net N$29: now also IC6.3; no longer IC6.2
- net N$3: now also C7.1, IC4.8, IC5.OUT; no longer IC1.10, U1.A7
- net N$30: now also U1.8; no longer U1.44
- net N$31: now also U1.A4; no longer U1.A5
- net N$33: now also IC1.7, U1.A9; no longer IC2.15, U1.A10
- net N$35: now also X3.2, X3.2@1, X3.2@2; no longer J1.BARREL, J1.SPRING
- net N$36: now also X4.2, X4.2@1, X4.2@2; no longer J2.BARREL, J2.SPRING
- net N$37: now also K1.S; no longer U$15.3
- net N$38: now also X5.2, X5.2@1, X5.2@2; no longer J3.BARREL, J3.SPRING
- net N$4: now also X2.1; no longer X2.3
- net N$45: now also IC4.14; no longer IC4.11
- net N$46: now also U1.30; no longer U1.26
- net N$48: now also IC1.10, U1.A8; no longer IC2.10, U1.A11
- net N$49: now also IC1.15, U1.A7; no longer IC2.7, U1.A12
- net N$50: now also IC1.2, U1.A6; no longer IC2.2, U1.A13
- net N$51: now also IC4.11; no longer IC4.14
- net N$53: now also JP1.4, U1.22; no longer JP1.9, U1.34
- net N$54: now also IC6.14, K4.1; no longer IC6.13, U$9.5
- net N$55: now also IC6.13, K5.1; no longer IC6.14, U$11.5
- net N$56: now also K3.1; no longer U$12.5
- net N$57: now also K2.1; no longer U$13.5
- net N$58: now also IC1.8, IC2.8; no longer IC1.16, IC2.16
- net N$59: now also JP2.6, U1.5; no longer TEMP.2, U1.6
- net N$6: now also X1.1; no longer X1.3
- net N$62: now also JP1.3, U1.23; no longer F7.P$2, U$13.3
- net N$63: now also K1.1; no longer U$15.5
- net N$64: now also X6.2, X6.2@1, X6.2@2; no longer J4.BARREL, J4.SPRING
- net N$65: now also JP2.4, U1.6; no longer TEMP1.2, U1.7
- net N$66: now also JP1.6, U1.24; no longer F6.P$2, U$12.3
- net N$67: now also JP1.5, U1.25; no longer F5.P$2, U$11.3
- net N$68: now also JP1.8, U1.26; no longer F4.P$2, U$9.3
- net N$70: now also JP1.7, U1.27; no longer JP1.8, U1.33
- net N$71: now also JP2.2, U1.7; no longer TEMP2.2, U1.8
- net N$72: now also JP1.10, U1.28; no longer JP1.7, U1.32
- net N$74: now also JP1.9, U1.29; no longer JP1.6, U1.31
- net N$8: now also F4.P$2, K2.S; no longer C7.1, IC4.16, IC5.OUT
- net N$9: now also F5.P$2, K3.S; no longer IC1.15, U1.A6
- net V+: now also K1.P; no longer U$15.2
Routing:
- net GND: track 0.00 -> 833.5 mm
- net +12V: track 0.00 -> 552.5 mm, vias 0 -> 1
- net +5V: track 0.00 -> 334.5 mm, vias 0 -> 2
- net N$12: track 0.00 -> 197.2 mm, vias 0 -> 4
- net N$40: track 0.00 -> 126.2 mm
- net N$41: track 0.00 -> 114.5 mm
- net N$32: track 0.00 -> 109.7 mm, vias 0 -> 6
- net N$42: track 0.00 -> 106.8 mm
- net N$23: track 0.00 -> 106.7 mm, vias 0 -> 1
- net N$44: track 0.00 -> 105.1 mm, vias 0 -> 1
- net N$39: track 0.00 -> 104.2 mm
- net N$58: track 0.00 -> 100.2 mm
- net V+: track 0.00 -> 99.8 mm
- net N$31: track 0.00 -> 94.0 mm, vias 0 -> 1
- net N$34: track 0.00 -> 92.5 mm, vias 0 -> 1
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Other:
- board size 191.8 x 149.9 mm -> 193 x 147.3 mm

Commit message: PCB fixes
Parts:
- removed JP2: RJ45, SparkFun-Connectors:RJ45-8
- removed U$6: SW motor, SparkFun:RJ9
- removed U$7: Hand control, SparkFun:RJ9
- added C5: 100n, SparkFun:CAP-PTH-5MM
- added F8: 6A, SparkFun:PTC
- added U$4, U$5: RJ9, jolo-lib:RJ9
- added U$8: RJ45, jolo-lib:RJ45
- F1, F2, F3: value PTCPTH -> 2A
- F4, F5, F6, F7: value PTCPTH -> 4A
- J5: value RJ11 -> COMM
- JP1: value (none) -> EXT
- X3: value TOBU3 -> PWM1
- X4: value TOBU3 -> PWM2
- X5: value TOBU3 -> PWM3
- X6: value TOBU3 -> PWM4
- moved C4 53.4 mm to (142.2, 94.0), turned to 270 degrees
- moved C3 10.9 mm to (114.3, 88.9), turned to 0 degrees
- moved Q1 2.54 mm to (115.6, 102.9), turned to 270 degrees
- moved Q4 2.54 mm to (100.3, 102.9), turned to 270 degrees
- moved F5 1.80 mm to (137.2, 88.9)
- moved Q3 1.27 mm to (146.1, 102.9), turned to 270 degrees
- moved F4 1.27 mm to (148.6, 88.9)
- turned Q2 to 270 degrees
Connections:
- new net N$75: IC1.1, IC1.9, U1.46
- new net N$76: C3.2, C4.1, F8.P$2, X3.1, X4.1, X5.1, X6.1
- net +12V: now also F8.P$1, U$3.Z1; no longer C3.1, C4.1, U$3.Z2, X3.1, X4.1, X5.1, X6.1
- net +5V: now also C5.2, U$5.4, U$8.1; no longer JP2.8, U$7.4
- net GND: now also C3.1, C5.1, U$5.1, U$8.2, U$8.4, U$8.6, U$8.8; no longer C3.2, JP2.1, JP2.3, JP2.5, JP2.7, U$7.1
- net N$1: now also R18.P$2, U1.21; no longer R17.P$2, U1.20
- net N$12: no longer IC1.1, IC1.9
- net N$2: now also R17.P$2, U1.20; no longer R18.P$2, U1.21
- net N$26: now also U$3.Z2; no longer U$3.Z1
- net N$34: now also U$5.2; no longer U$7.2
- net N$44: now also U$5.3; no longer U$7.3
- net N$45: now also U$4.3, U$4.4; no longer U$6.3, U$6.4
- net N$51: now also U$4.1, U$4.2; no longer U$6.1, U$6.2
- net N$59: now also U$8.7; no longer JP2.6
- net N$65: now also U$8.5; no longer JP2.4
- net N$71: now also U$8.3; no longer JP2.2
Routing:
- net +5V: track 334.5 -> 492.8 mm
- net N$75: track 0.00 -> 135.5 mm, vias 0 -> 2
- net N$76: track 0.00 -> 125.2 mm
- net +12V: track 552.5 -> 467.3 mm, vias 1 -> 0
- net GND: track 833.5 -> 868.0 mm
- net N$12: track 197.2 -> 164.1 mm, vias 4 -> 3
- net N$46: track 56.7 -> 73.6 mm, vias 0 -> 1
- net N$42: track 106.8 -> 97.0 mm, vias 0 -> 1
- net N$69: track 18.4 -> 24.7 mm
- net N$35: track 9.21 -> 15.5 mm
- net N$52: track 18.9 -> 25.0 mm
- net N$41: track 114.5 -> 108.4 mm, vias 0 -> 1
- net N$59: track 52.3 -> 58.4 mm
- net N$1: track 42.4 -> 48.4 mm
- net N$31: track 94.0 -> 99.9 mm
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- added copper zone on layer 16, net +12V
- added copper zone on layer 1, net GND
Other:
- board size 193 x 147.3 mm -> 167.6 x 124.5 mm
- board text added: "12V input"
- board text added: "12V outputs"
- board text added: "22"
- board text added: "24"
- board text added: "26"
- board text added: "28"
- board text added: "5V"
- board text added: "AstroHub 3.0"
- board text added: "COMM"
- board text added: "DC motor"
- board text added: "GND"
- board text added: "Hand controller"
- board text added: "PWM outputs"
- board text added: "SENSORS"
- board text added: "STEPPER 1"
- board text added: "STEPPER 2"
- board text added: "V reg"
- board text added: "astrojolo.blogspot.com 2015.07"
